Commit message: Implement Gazebo Thruster plugin system for realistic propeller physics
Major changes:
- Convert thruster joints from fixed to revolute (Y-axis rotation)
- Add Gazebo Sim 8 Thruster plugins for left and right propellers
- Update thrust controller to publish angular velocity commands instead of wrench
- Add ROS2->Gazebo Transport bridge for thruster command topics
- Fix NaN handling in guidance tracker with timing safeguards
- Set wind velocity to 0 for initial thrust testing

Technical details:
- Thruster plugins use default topic pattern: /model/marid/joint/{joint_name}/cmd_vel
- Angular velocity conversion: omega = gain * sqrt(thrust)
- Added timing safeguards in PID controllers to handle system lag
- Bridge syntax: ] for ROS2->Gazebo, [ for Gazebo->ROS2

Status: Thrust is now being applied and drone moves, but still unstable.
Next steps: Tune joint axis direction, enable gravity, adjust thrust coefficients.

File: src/marid_description/urdf/marid.urdf.xacro (robot description, xacro)
@@ -299,13 +299,19 @@
       <collision><origin xyz="0 0 0"/><geometry><cylinder length="0.1" radius="0.015"/></geometry></collision>
   </link>
-  <joint name="thruster_L_joint" type="fixed">
+  <joint name="thruster_L_joint" type="revolute">
     <parent link="base_link_front"/>
     <child  link="thruster_L"/>
     <origin xyz="-0.30  0.20 -0.05" rpy="0 0 0"/>
-  </joint>
-  <joint name="thruster_R_joint" type="fixed">
+    <axis xyz="0 1 0"/>  <!-- Rotate around Y-axis (forward direction) -->
+    <limit lower="-3.14159" upper="3.14159" effort="100" velocity="100"/>
+    <dynamics damping="0.01" friction="0.0"/>
+  </joint>
+  <joint name="thruster_R_joint" type="revolute">
     <parent link="base_link_front"/>
     <child  link="thruster_R"/>
     <origin xyz="0.30 0.20 -0.05" rpy="0 0 0"/>
+    <axis xyz="0 1 0"/>  <!-- Rotate around Y-axis (forward direction) -->
+    <limit lower="-3.14159" upper="3.14159" effort="100" velocity="100"/>
+    <dynamics damping="0.01" friction="0.0"/>
   </joint>
 </robot>

File: src/marid_description/urdf/marid_gazebo.xacro (robot description, xacro)
@@ -52,4 +52,29 @@
     </gazebo>
     <gazebo>
+        <plugin name="lifting_surface" filename="libLiftDragPlugin.so">
+        <!-- taken from the lift curve figure -->
+        <!-- alpha_0 is 5 degrees -->
+        <a0>0.08727</a0>
+        <!-- alpha_stall is 19.3 degrees -->
+        <alpha_stall>0.3368</alpha_stall>
+        <!-- slope of the lift curve to the left of the stall angle -->
+        <cla>5.418</cla>
+        <!-- slope of the lift curve to the right of the stall angle -->
+        <cla_stall>-2.1419</cla_stall>
+        <!-- below are just random values in this example -->
+        <cda>0.0</cda>
+        <cda_stall>0.0</cda_stall>
+        <cma>0.0</cma>
+        <cma_stall>0.0</cma_stall>
+        <area>3</area>
+        <fluid_density>1.2041</fluid_density>
+        <forward>-1 0 0</forward>
+        <upward>0 -1 0</upward>
+        <cp>0 0 1</cp>
+        <link_name>lifting_surface_link</link_name>
+        <radial_symmetry>false</radial_symmetry>
+      </plugin>
+    </gazebo>
+    <gazebo>
         <plugin filename="libgz-sim8-lift-drag-system.so" name="gz::sim::systems::LiftDrag">
             <link_name>right_wing</link_name>
@@ -127,4 +152,28 @@
             <cp>0 0 0</cp>  <!-- No offset for tail -->
             <debug>true</debug>
+        </plugin>
+    </gazebo>
+    <!-- ===== THRUSTER PLUGINS ===== -->
+    <!-- Left Thruster -->
+    <!-- Gazebo Sim 8 Thruster plugin uses default topic: /model/{namespace}/joint/{joint_name}/cmd_vel -->
+    <gazebo>
+        <plugin filename="libgz-sim8-thruster-system.so" name="gz::sim::systems::Thruster">
+            <namespace>marid</namespace>
+            <joint_name>thruster_L_joint</joint_name>
+            <fluid_density>1.225</fluid_density>  <!-- Air density at sea level (kg/m³) -->
+            <propeller_diameter>0.2</propeller_diameter>  <!-- Adjust based on your propeller size (meters) -->
+            <thrust_coefficient>0.8</thrust_coefficient>  <!-- Typical range: 0.6-1.0 -->
+            <use_angvel_cmd>true</use_angvel_cmd>  <!-- Accept angular velocity commands (rad/s) -->
+        </plugin>
+    </gazebo>
+    <!-- Right Thruster -->
+    <gazebo>
+        <plugin filename="libgz-sim8-thruster-system.so" name="gz::sim::systems::Thruster">
+            <namespace>marid</namespace>
+            <joint_name>thruster_R_joint</joint_name>
+            <fluid_density>1.225</fluid_density>
+            <propeller_diameter>0.2</propeller_diameter>
+            <thrust_coefficient>0.8</thrust_coefficient>
+            <use_angvel_cmd>true</use_angvel_cmd>
         </plugin>
     </gazebo>

Commit message: Fix Gazebo integration and improve control system stability
- Fixed XML parsing errors and NaN handling in thrust calculations
- Corrected Gazebo plugin configuration (Thruster, JointPositionController)
- Added ros_gz_bridge for thruster and joint command topics
- Fixed attitude controller for Y-forward orientation (swapped roll/pitch)
- Added center thruster option and thrust smoothing/rate limiting
- Adjusted control parameters and inertia tensors for stability
- Zeroed wind/gravity for controlled testing

Testing: Simulation launches and responds to commands (stability tuning ongoing)

File: src/marid_description/urdf/marid.urdf.xacro (robot description, xacro)
@@ -20,6 +20,6 @@
     <inertial>
       <mass value="3.0903248"/>
-      <origin xyz="0 0.1 0.02" rpy="0 0 0"/>
-      <inertia ixx="0.1110930358" ixy="0.0" ixz="0.0" iyy="0.0247075659" iyz="0.0027559088" izz="0.1288539854"/>
+      <origin xyz="0 0 0" rpy="0 0 0"/>  <!-- Fixed: COM at geometric center for stability -->
+      <inertia ixx="0.1110930358" ixy="0.0" ixz="0.0" iyy="0.0247075659" iyz="0.0" izz="0.1288539854"/>  <!-- Fixed: Zeroed iyz to eliminate cross-coupling moments -->
     </inertial>
     <visual>
@@ -302,6 +302,6 @@
     <parent link="base_link_front"/>
     <child  link="thruster_L"/>
-    <origin xyz="-0.30  0.20 -0.05" rpy="0 0 0"/>
-    <axis xyz="0 1 0"/>  <!-- Rotate around Y-axis (forward direction) -->
+    <origin xyz="-0.15 0.0 -0.02" rpy="0 0 0"/>  <!-- Fixed: Moved closer to COM to reduce moments -->
+    <axis xyz="0 1 0"/>  <!-- Reverted: Original axis was correct -->
     <limit lower="-3.14159" upper="3.14159" effort="100" velocity="100"/>
     <dynamics damping="0.01" friction="0.0"/>
@@ -310,8 +310,32 @@
     <parent link="base_link_front"/>
     <child  link="thruster_R"/>
-    <origin xyz="0.30 0.20 -0.05" rpy="0 0 0"/>
-    <axis xyz="0 1 0"/>  <!-- Rotate around Y-axis (forward direction) -->
+    <origin xyz="0.15 0.0 -0.02" rpy="0 0 0"/>  <!-- Fixed: Moved closer to COM to reduce moments -->
+    <axis xyz="0 1 0"/>  <!-- Reverted: Original axis was correct -->
     <limit lower="-3.14159" upper="3.14159" effort="100" velocity="100"/>
     <dynamics damping="0.01" friction="0.0"/>
   </joint>
+  <!-- Center Thruster (for single-thruster testing) -->
+  <link name="thruster_center">
+    <inertial>
+      <origin xyz="0 0 0" rpy="1.5708 0 0"/>
+      <mass value="0.05"/>
+      <inertia ixx="1e-5" ixy="0" ixz="0" iyy="1e-5" iyz="0" izz="1e-5"/>
+    </inertial>
+    <visual>
+      <origin xyz="0 0 0" rpy="1.5708 0 0"/>
+      <geometry><cylinder length="0.1" radius="0.015"/></geometry>
+      <material name="green_thruster">
+        <color rgba="0.0 1.0 0.0 1.0"/>
+      </material>
+    </visual>
+    <collision><origin xyz="0 0 0" rpy="1.5708 0 0"/><geometry><cylinder length="0.1" radius="0.015"/></geometry></collision>
+  </link>
+  <joint name="thruster_center_joint" type="revolute">
+    <parent link="base_link_front"/>
+    <child link="thruster_center"/>
+    <origin xyz="0.0 0.0 0.0" rpy="0 0 0"/>  <!-- At COM - no moments -->
+    <axis xyz="0 1 0"/>
+    <limit lower="-3.14159" upper="3.14159" effort="100" velocity="100"/>
+    <dynamics damping="0.01" friction="0.0"/>
+  </joint>
 </robot>

File: src/marid_description/urdf/marid_gazebo.xacro (robot description, xacro)
@@ -52,29 +52,4 @@
     </gazebo>
     <gazebo>
-        <plugin name="lifting_surface" filename="libLiftDragPlugin.so">
-        <!-- taken from the lift curve figure -->
-        <!-- alpha_0 is 5 degrees -->
-        <a0>0.08727</a0>
-        <!-- alpha_stall is 19.3 degrees -->
-        <alpha_stall>0.3368</alpha_stall>
-        <!-- slope of the lift curve to the left of the stall angle -->
-        <cla>5.418</cla>
-        <!-- slope of the lift curve to the right of the stall angle -->
-        <cla_stall>-2.1419</cla_stall>
-        <!-- below are just random values in this example -->
-        <cda>0.0</cda>
-        <cda_stall>0.0</cda_stall>
-        <cma>0.0</cma>
-        <cma_stall>0.0</cma_stall>
-        <area>3</area>
-        <fluid_density>1.2041</fluid_density>
-        <forward>-1 0 0</forward>
-        <upward>0 -1 0</upward>
-        <cp>0 0 1</cp>
-        <link_name>lifting_surface_link</link_name>
-        <radial_symmetry>false</radial_symmetry>
-      </plugin>
-    </gazebo>
-    <gazebo>
         <plugin filename="libgz-sim8-lift-drag-system.so" name="gz::sim::systems::LiftDrag">
             <link_name>right_wing</link_name>
@@ -139,5 +114,5 @@
         </plugin>
     </gazebo>
-    <gazebo>
+    <gazebo reference="main_tail">
         <plugin filename="libgz-sim8-lift-drag-system.so" name="gz::sim::systems::LiftDrag">
             <link_name>main_tail</link_name>
@@ -176,4 +151,52 @@
             <thrust_coefficient>0.8</thrust_coefficient>
             <use_angvel_cmd>true</use_angvel_cmd>
+        </plugin>
+    </gazebo>
+    <!-- Center Thruster (for single-thruster testing) -->
+    <gazebo>
+        <plugin filename="libgz-sim8-thruster-system.so" name="gz::sim::systems::Thruster">
+            <namespace>marid</namespace>
+            <joint_name>thruster_center_joint</joint_name>
+            <fluid_density>1.225</fluid_density>
+            <propeller_diameter>0.2</propeller_diameter>
+            <thrust_coefficient>0.8</thrust_coefficient>
+            <use_angvel_cmd>true</use_angvel_cmd>
+        </plugin>
+    </gazebo>
+    <!-- ===== JOINT POSITION CONTROLLERS FOR CONTROL SURFACES ===== -->
+    <!-- Left Wing Position Controller -->
+    <gazebo>
+        <plugin filename="libgz-sim8-joint-position-controller-system.so"
+                name="gz::sim::systems::JointPositionController">
+            <joint_name>left_wing_joint</joint_name>
+            <p_gain>0.5</p_gain>  <!-- Increased from 0.1 for faster control surface response -->
+            <topic>/model/marid/joint/left_wing_joint/cmd_pos</topic>
+        </plugin>
+    </gazebo>
+    <!-- Right Wing Position Controller -->
+    <gazebo>
+        <plugin filename="libgz-sim8-joint-position-controller-system.so"
+                name="gz::sim::systems::JointPositionController">
+            <joint_name>right_wing_joint</joint_name>
+            <p_gain>0.5</p_gain>  <!-- Increased from 0.1 for faster control surface response -->
+            <topic>/model/marid/joint/right_wing_joint/cmd_pos</topic>
+        </plugin>
+    </gazebo>
+    <!-- Left Tail Position Controller -->
+    <gazebo>
+        <plugin filename="libgz-sim8-joint-position-controller-system.so"
+                name="gz::sim::systems::JointPositionController">
+            <joint_name>tail_left_joint</joint_name>
+            <p_gain>0.5</p_gain>  <!-- Increased from 0.1 for faster control surface response -->
+            <topic>/model/marid/joint/tail_left_joint/cmd_pos</topic>
+        </plugin>
+    </gazebo>
+    <!-- Right Tail Position Controller -->
+    <gazebo>
+        <plugin filename="libgz-sim8-joint-position-controller-system.so"
+                name="gz::sim::systems::JointPositionController">
+            <joint_name>tail_right_joint</joint_name>
+            <p_gain>0.5</p_gain>  <!-- Increased from 0.1 for faster control surface response -->
+            <topic>/model/marid/joint/tail_right_joint/cmd_pos</topic>
         </plugin>
     </gazebo>

Commit message: Fix thruster reaction torque by removing joint damping
Reduced damping on thruster_center_joint from 2.0 to 0.0 to allow
reaction torque to be properly visible. High damping was preventing
the body from rotating in response to propeller reaction torque,
making it appear as if the propeller was locked to the body.

With zero damping, the drone now correctly exhibits opposite rotation
to the propeller direction, demonstrating proper reaction torque physics.

File: src/marid_description/urdf/marid.urdf.xacro (robot description, xacro)
@@ -318,10 +318,10 @@
   <link name="thruster_center">
     <inertial>
-      <origin xyz="0 0 0" rpy="1.5708 0 0"/>
-      <mass value="0.05"/>
-      <inertia ixx="1e-5" ixy="0" ixz="0" iyy="1e-5" iyz="0" izz="1e-5"/>
-    </inertial>
-    <visual>
-      <origin xyz="0 0 0" rpy="1.5708 0 0"/>
+      <origin xyz="0 0 0" rpy="1.5708 0 0"/>  <!-- Rotate 90° around X so local Z aligns with body Y (forward direction) -->
+      <mass value="0.05"/>  <!-- Increased from 0.001 to 0.05 for better stability -->
+      <inertia ixx="5e-4" ixy="0" ixz="0" iyy="5e-4" iyz="0" izz="5e-4"/>  <!-- Scaled with mass -->
+    </inertial>
+    <visual>
+      <origin xyz="0 0 0" rpy="1.5708 0 0"/>  <!-- Rotation only in visual -->
       <geometry><cylinder length="0.1" radius="0.015"/></geometry>
       <material name="green_thruster">
@@ -329,5 +329,5 @@
       </material>
     </visual>
-    <collision><origin xyz="0 0 0" rpy="1.5708 0 0"/><geometry><cylinder length="0.1" radius="0.015"/></geometry></collision>
+    <!-- NO COLLISION - prevents overlap issues, thruster is visual-only and force application doesn't need collision -->
   </link>
   <joint name="thruster_center_joint" type="revolute">
@@ -336,6 +336,6 @@
     <origin xyz="0.0 0.0 0.0" rpy="0 0 0"/>  <!-- At COM - no moments -->
     <axis xyz="0 1 0"/>
-    <limit lower="-3.14159" upper="3.14159" effort="100" velocity="100"/>
-    <dynamics damping="0.01" friction="0.0"/>
+    <limit lower="-1000" upper="1000" effort="1000" velocity="1000"/>  <!-- Very loose limits for unlimited rotation -->
+    <dynamics damping="0.0" friction="0.0"/>  <!-- Zero damping to allow full reaction torque visibility -->
   </joint>
 </robot>

File: src/marid_description/urdf/marid_gazebo.xacro (robot description, xacro)
@@ -112,4 +112,33 @@
             <cp>0 0 0</cp>  <!-- No offset for fuselage -->
             <debug>true</debug>
+        </plugin>
+    </gazebo>
+    <!-- Aerodynamic Damping for Main Body (prevents uncontrolled rotations and drift) -->
+    <gazebo reference="base_link_front">
+        <plugin filename="libgz-sim8-hydrodynamics-system.so"
+                name="gz::sim::systems::Hydrodynamics">
+            <link_name>base_link_front</link_name>
+            <!-- Linear drag coefficients (X, Y, Z) - acts like air resistance -->
+            <xDotU>-0.5</xDotU>    <!-- Forward drag (X-axis) -->
+            <yDotV>-1.0</yDotV>    <!-- Side drag (Y-axis - your forward) -->
+            <zDotW>-1.0</zDotW>    <!-- Vertical drag (Z-axis) -->
+            <!-- Angular drag coefficients (Roll, Pitch, Yaw) - rotational damping -->
+            <kDotP>-2.0</kDotP>    <!-- Roll damping (around X) -->
+            <mDotQ>-2.0</mDotQ>     <!-- Pitch damping (around Y) -->
+            <nDotR>-2.0</nDotR>     <!-- Yaw damping (around Z) -->
+            <!-- Quadratic drag (velocity-squared terms) -->
+            <xUabsU>-0.1</xUabsU>   <!-- Forward quadratic drag -->
+            <yVabsV>-0.2</yVabsV>   <!-- Side quadratic drag -->
+            <zWabsW>-0.2</zWabsW>   <!-- Vertical quadratic drag -->
+            <kPabsP>-1.0</kPabsP>  <!-- Roll quadratic damping -->
+            <mQabsQ>-1.0</mQabsQ>  <!-- Pitch quadratic damping -->
+            <nRabsR>-1.0</nRabsR>  <!-- Yaw quadratic damping -->
+            <!-- Linear velocity terms (usually zero for air) -->
+            <xU>0</xU>
+            <yV>0</yV>
+            <zW>0</zW>
+            <kP>0</kP>
+            <mQ>0</mQ>
+            <nR>0</nR>
         </plugin>
     </gazebo>
