Commit message: Localization: - Fix gazebo_pose_to_odom gz model output parsing - Update map→odom TF and offset handling
Controllers:
- Increase controller spawner timeout to 120s for reliable startup

File: src/marid_description/urdf/marid.urdf.xacro (robot description, xacro)
@@ -154,5 +154,5 @@
     <parent link="main_tail"/>
     <child link="tail_left"/>
-    <origin xyz="0 -.28 0" rpy="0.3491 0 0"/>
+    <origin xyz="0 -.28 0" rpy="0 0 0"/>
     <axis xyz="0.7071 0 -0.7071"/>
     <dynamics damping="2.5" friction="1.0"/>  <!-- Reduced for servo-like behavior: locked when idle, moves when commanded -->
@@ -189,5 +189,5 @@
     <parent link="main_tail"/>
     <child link="tail_right"/>
-    <origin xyz="0 -0.28 0" rpy="0.3491 0 0"/>
+    <origin xyz="0 -0.28 0" rpy="0 0 0"/>
     <axis xyz="0.7071 0 0.7071"/>
     <dynamics damping="2.5" friction="1.0"/>  <!-- Reduced for servo-like behavior: locked when idle, moves when commanded -->

File: src/marid_description/urdf/marid_gazebo.xacro (robot description, xacro)
@@ -287,11 +287,12 @@
         <gz_frame_id>gps_link</gz_frame_id>
         <!-- GPS Noise Model (realistic consumer-grade GPS) -->
+        <!-- WARNING: gz-sensors NavSat treats stddev as DEGREES not meters (bug #325). -->
+        <!-- Use 0.00002 ≈ 2.2m at 37°N; 2.5 would add ±2.5° ≈ ±280km noise. -->
         <navsat>
-          <!-- Horizontal position noise (standard deviation in meters) -->
           <position_sensing>
             <horizontal>
               <noise type="gaussian">
                 <mean>0.0</mean>
-                <stddev>2.5</stddev> <!-- 2m horizontal accuracy (consumer GPS) -->
+                <stddev>0.00002</stddev> <!-- ~2.5m equiv (workaround for degrees bug) -->
               </noise>
             </horizontal>
@@ -299,5 +300,5 @@
               <noise type="gaussian">
                 <mean>0.0</mean>
-                <stddev>2.5</stddev> <!-- 4m vertical accuracy (worse than horizontal) -->
+                <stddev>0.00002</stddev> <!-- ~2.5m equiv (workaround for degrees bug) -->
               </noise>
             </vertical>

Commit message: Add Madgwick IMU orientation pipeline for EKF
- imu_filter_madgwick fuses gyro+accel -> orientation; republisher feeds /imu_ekf
- imu_add_gravity adds world gravity in body frame (using /imu/data feedback) so Madgwick works with Gazebo's specific-force IMU in sim and on real hardware
- EKF uses orientation from filtered IMU; config and launch wiring

File: src/marid_description/urdf/marid.urdf.xacro (robot description, xacro)
@@ -73,4 +73,7 @@
         <mesh filename="package://marid_description/meshes/left_wing.stl"/>
       </geometry>
+      <material name="left_wing_red">
+        <color rgba="1.0 0.0 0.0 1.0"/>
+      </material>
     </visual>
     <collision>
@@ -108,4 +111,7 @@
         <mesh filename="package://marid_description/meshes/right_wing.stl"/>
       </geometry>
+      <material name="right_wing_blue">
+        <color rgba="0.0 0.0 1.0 1.0"/>
+      </material>
     </visual>
     <collision>
@@ -143,4 +149,7 @@
         <mesh filename="package://marid_description/meshes/tail_left.stl"/>
       </geometry>
+      <material name="tail_left_red">
+        <color rgba="1.0 0.0 0.0 1.0"/>
+      </material>
     </visual>
     <collision>
@@ -178,4 +187,7 @@
         <mesh filename="package://marid_description/meshes/tail_right.stl"/>
       </geometry>
+      <material name="tail_right_blue">
+        <color rgba="0.0 0.0 1.0 1.0"/>
+      </material>
     </visual>
     <collision>

File: src/marid_description/urdf/marid_gazebo.xacro (robot description, xacro)
@@ -237,4 +237,5 @@
           <topic>/imu</topic>
           <imu>
+            <enable_orientation>true</enable_orientation>
             <angular_velocity>
               <x>

Commit message: Temporary setup: use Gazebo OdometryPublisher for simulation odometry until marid_odom_pub (marid_controller) is fixed and robust enough to serve as the main pose source.
- Add OdometryPublisher plugin to MARID model (marid_gazebo.xacro) to
  publish ground-truth odometry on /model/marid/odometry (pose + twist,
  publish_tf: false).
- Bridge /model/marid/odometry to /gazebo/odom in gazebo.launch.py for
  the local EKF.
- Use orientation from /gazebo/odom in local EKF (odom0_config) to avoid
  IMU-only orientation drift in simulation.
- Remove gazebo_pose_to_odom node (broken world pose topics), delete
  script, drop from launch and CMakeLists, and update marid_logging README.

File: src/marid_description/urdf/marid.urdf.xacro (robot description, xacro)
@@ -17,4 +17,13 @@
   <xacro:property name="right_wing_offset" value="0.0 ${-axis_offset_y} 0.0"/>
   <xacro:property name="wing_axis" value="1 0 0"/>
+  <!-- Spawn height: whole robot is lifted so it spawns above ground when model origin is at (0,0,0) -->
+  <xacro:property name="spawn_z_offset" value="0.12"/>
+  <!-- Root link at model origin (spawn point). No geometry/inertial needed. -->
+  <link name="base_footprint"/>
+  <joint name="base_footprint_joint" type="fixed">
+    <parent link="base_footprint"/>
+    <child link="base_link_front"/>
+    <origin xyz="0 0 ${spawn_z_offset}" rpy="0 0 0"/>
+  </joint>
   <link name="base_link_front">
     <inertial>
@@ -319,4 +328,5 @@
       <inertia ixx="1e-5" ixy="0" ixz="0" iyy="1e-5" iyz="0" izz="1e-5"/>
       </inertial>
+      <!-- Hub/center cylinder -->
       <visual>
         <origin xyz="0 0 0" rpy="1.5708 0 0"/><geometry><cylinder length="0.1" radius="0.015"/></geometry>
@@ -325,4 +335,36 @@
         </material>
       </visual>
+      <!-- Propeller blade 1 - visible indicator for rotation -->
+      <visual>
+        <origin xyz="0.08 0 0" rpy="1.5708 0 0"/>
+        <geometry><box size="0.15 0.01 0.02"/></geometry>
+        <material name="red_thruster">
+          <color rgba="1.0 0.3 0.3 1.0"/>
+        </material>
+      </visual>
+      <!-- Propeller blade 2 - opposite side -->
+      <visual>
+        <origin xyz="-0.08 0 0" rpy="1.5708 0 0"/>
+        <geometry><box size="0.15 0.01 0.02"/></geometry>
+        <material name="red_thruster">
+          <color rgba="1.0 0.3 0.3 1.0"/>
+        </material>
+      </visual>
+      <!-- Propeller blade 3 - perpendicular -->
+      <visual>
+        <origin xyz="0 0.08 0" rpy="1.5708 0 0"/>
+        <geometry><box size="0.01 0.15 0.02"/></geometry>
+        <material name="red_thruster">
+          <color rgba="1.0 0.3 0.3 1.0"/>
+        </material>
+      </visual>
+      <!-- Propeller blade 4 - opposite -->
+      <visual>
+        <origin xyz="0 -0.08 0" rpy="1.5708 0 0"/>
+        <geometry><box size="0.01 0.15 0.02"/></geometry>
+        <material name="red_thruster">
+          <color rgba="1.0 0.3 0.3 1.0"/>
+        </material>
+      </visual>
       <collision><origin xyz="0 0 0"/><geometry><cylinder length="0.1" radius="0.015"/></geometry></collision>
   </link>
@@ -333,7 +375,42 @@
       <inertia ixx="1e-5" ixy="0" ixz="0" iyy="1e-5" iyz="0" izz="1e-5"/>
       </inertial>
-      <visual><origin xyz="0 0 0" rpy="1.5708 0 0"/><geometry><cylinder length="0.1" radius="0.015"/></geometry>
+      <!-- Hub/center cylinder -->
+      <visual>
+        <origin xyz="0 0 0" rpy="1.5708 0 0"/>
+        <geometry><cylinder length="0.1" radius="0.015"/></geometry>
         <material name="blue_thruster">
           <color rgba="0.0 0.0 1.0 1.0"/>
+        </material>
+      </visual>
+      <!-- Propeller blade 1 - visible indicator for rotation -->
+      <visual>
+        <origin xyz="0.08 0 0" rpy="1.5708 0 0"/>
+        <geometry><box size="0.15 0.01 0.02"/></geometry>
+        <material name="blue_thruster">
+          <color rgba="0.3 0.3 1.0 1.0"/>
+        </material>
+      </visual>
+      <!-- Propeller blade 2 - opposite side -->
+      <visual>
+        <origin xyz="-0.08 0 0" rpy="1.5708 0 0"/>
+        <geometry><box size="0.15 0.01 0.02"/></geometry>
+        <material name="blue_thruster">
+          <color rgba="0.3 0.3 1.0 1.0"/>
+        </material>
+      </visual>
+      <!-- Propeller blade 3 - perpendicular -->
+      <visual>
+        <origin xyz="0 0.08 0" rpy="1.5708 0 0"/>
+        <geometry><box size="0.01 0.15 0.02"/></geometry>
+        <material name="blue_thruster">
+          <color rgba="0.3 0.3 1.0 1.0"/>
+        </material>
+      </visual>
+      <!-- Propeller blade 4 - opposite -->
+      <visual>
+        <origin xyz="0 -0.08 0" rpy="1.5708 0 0"/>
+        <geometry><box size="0.01 0.15 0.02"/></geometry>
+        <material name="blue_thruster">
+          <color rgba="0.3 0.3 1.0 1.0"/>
         </material>
       </visual>
@@ -352,5 +429,5 @@
     <child  link="thruster_R"/>
     <origin xyz="0.15 0.0 -0.02" rpy="0 0 0"/>
-    <axis xyz="0 1 0"/>  <!-- Reverted: Original axis was correct -->
+    <axis xyz="0 1 0"/>  <!-- Normal axis: both axes same, counter-rotation via negative angular velocity -->
     <!-- Continuous joints don't have limits - unlimited rotation for propellers -->
     <dynamics damping="0.0" friction="0.0"/>  <!-- Zero damping to allow full reaction torque visibility -->

File: src/marid_description/urdf/marid_gazebo.xacro (robot description, xacro)
@@ -178,5 +178,5 @@
             <fluid_density>1.225</fluid_density>
             <propeller_diameter>0.2</propeller_diameter>
-            <thrust_coefficient>0.8</thrust_coefficient>  <!-- Positive coefficient - counter-rotation achieved via reversed joint axis -->
+            <thrust_coefficient>0.8</thrust_coefficient>  <!-- Typical range: 0.6-1.0 -->
             <use_angvel_cmd>true</use_angvel_cmd>
         </plugin>
@@ -427,4 +427,13 @@
       </plugin>
     </gazebo>
+    <!-- Odometry Publisher - ground-truth odom for EKF (pose + twist in odom frame) -->
+    <gazebo>
+      <plugin filename="gz-sim-odometry-publisher-system" name="gz::sim::systems::OdometryPublisher">
+        <odom_topic>/model/marid/odometry</odom_topic>
+        <odom_frame>odom</odom_frame>
+        <robot_base_frame>base_link_front</robot_base_frame>
+        <publish_tf>false</publish_tf>
+      </plugin>
+    </gazebo>
         <!-- Camera for perception / ML -->
     <gazebo reference="camera_link">
