Commit message: Provisional landing gear for ground testing (drone is provisional CAD).
Landing gear:
- Add left/right front wheel arms and rear wheel arm with CAD-derived inertials
  and joint positions (arm attachment xyz from CAD; z negative below origin).
- Add revolute (continuous) wheel joints for all three wheels; rotation axis
  aligned with world X (wheel axle); joint/link z offsets tuned for wheel axis.
- Add rear wheel link and rear_wheel_joint; rear arm attached on centerline.
- Use wheel.stl, front_wheel_arm.stl, rear_wheel_arm.stl for visuals/collision.

Controller / launch:
- Default to center thruster and 10 N initial thrust (option_a).
- Spawn at z = 1 m from gazebo.launch.py (-z 1.0); revert spawn_z_offset in URDF.
- Remove visuals for left/right thrusters (thruster_L, thruster_R).

Inertials:
- Front/rear arm and wheel inertials from CAD or disk approximation; arm CoM
  and inertia tensor set from CAD data.

File: src/marid_description/urdf/marid.urdf.xacro (robot description, xacro)
@@ -45,4 +45,159 @@
     </collision>
   </link>
+  <!--Landing Gears-->
+  <link name="left_front_wheel_arm">
+    <inertial>
+      <mass value="0.005443"/>
+      <origin xyz="0 0 -0.069215" rpy="0 0 0"/>  <!-- CoM from CAD (front_wheel_arm), Z in m -->
+      <inertia ixx="1.756e-6" ixy="0" ixz="0" iyy="2.048e-6" iyz="0" izz="2.926e-7"/>  <!-- From CAD, kg⋅m² -->
+    </inertial>
+    <visual>
+      <origin xyz="0 0 0" rpy="0 0 0"/>
+      <geometry>
+        <mesh filename="package://marid_description/meshes/front_wheel_arm.stl"/>
+      </geometry>
+    </visual>
+    <collision>
+      <origin xyz="0 0 0" rpy="0 0 0"/>
+      <geometry>
+        <mesh filename="package://marid_description/meshes/front_wheel_arm.stl"/>
+      </geometry>
+    </collision>
+  </link>
+  <joint name="left_arm_joint" type="fixed">
+    <parent link="base_link_front"/>
+    <child link="left_front_wheel_arm"/>
+    <origin xyz="-0.053 0.355 -0.069" rpy="0 0 0"/>  <!-- Top of left arm from CAD (min dist), m; Z neg = below origin -->
+    <axis xyz="0 1 0"/>
+    <limit lower="0" upper="0" effort="1000" velocity="1000"/>
+  </joint>
+  <link name="right_front_wheel_arm">
+    <inertial>
+      <mass value="0.005443"/>
+      <origin xyz="0 0 -0.069215" rpy="0 0 0"/>  <!-- CoM from CAD (front_wheel_arm), Z in m -->
+      <inertia ixx="1.756e-6" ixy="0" ixz="0" iyy="2.048e-6" iyz="0" izz="2.926e-7"/>  <!-- From CAD, kg⋅m² -->
+    </inertial>
+    <visual>
+      <origin xyz="0 0 0" rpy="0 0 0"/>
+      <geometry>
+        <mesh filename="package://marid_description/meshes/front_wheel_arm.stl"/>
+      </geometry>
+    </visual>
+    <collision>
+      <origin xyz="0 0 0" rpy="0 0 0"/>
+      <geometry>
+        <mesh filename="package://marid_description/meshes/front_wheel_arm.stl"/>
+      </geometry>
+    </collision>
+  </link>
+  <joint name="right_arm_joint" type="fixed">
+    <parent link="base_link_front"/>
+    <child link="right_front_wheel_arm"/>
+    <origin xyz="0.053 0.355 -0.069" rpy="0 0 0"/>  <!-- Top of right arm from CAD (min dist), m; Z neg = below origin -->
+    <axis xyz="0 1 0"/>
+    <limit lower="0" upper="0" effort="1000" velocity="1000"/>
+  </joint>
+  <link name="left_front_wheel">
+    <inertial>
+      <mass value="0.05"/>  <!-- ~50 g, small landing wheel -->
+      <origin xyz="0 0 0" rpy="0 0 0"/>
+      <inertia ixx="7.8e-6" ixy="0" ixz="0" iyy="1.56e-5" iyz="0" izz="7.8e-6"/>  <!-- Disk r~0.025 m: I_ax=0.5*m*r^2, I_rad=0.25*m*r^2 -->
+    </inertial>
+    <visual>
+      <origin xyz="0 0 0.1016358" rpy="0 0 0"/>
+      <geometry>
+        <mesh filename="package://marid_description/meshes/wheel.stl"/>
+      </geometry>
+    </visual>
+    <collision>
+      <origin xyz="0 0 0.1016358" rpy="0 0 0"/>
+      <geometry>
+        <mesh filename="package://marid_description/meshes/wheel.stl"/>
+      </geometry>
+    </collision>
+  </link>
+  <joint name="left_front_wheel_joint" type="continuous">
+    <parent link="left_front_wheel_arm"/>
+    <child link="left_front_wheel"/>
+    <origin xyz="0 0 -0.1016358" rpy="0 0 0"/>
+    <axis xyz="1 0 0"/>  <!-- Wheel rotation around own axle (parallel to world X) -->
+    <dynamics damping="0.01" friction="0.0"/>
+  </joint>
+  <link name="right_front_wheel">
+    <inertial>
+      <mass value="0.05"/>  <!-- ~50 g, small landing wheel -->
+      <origin xyz="0 0 0" rpy="0 0 0"/>
+      <inertia ixx="7.8e-6" ixy="0" ixz="0" iyy="1.56e-5" iyz="0" izz="7.8e-6"/>  <!-- Disk r~0.025 m: I_ax=0.5*m*r^2, I_rad=0.25*m*r^2 -->
+    </inertial>
+    <visual>
+      <origin xyz="0 0 0.1016358" rpy="0 0 0"/>
+      <geometry>
+        <mesh filename="package://marid_description/meshes/wheel.stl"/>
+      </geometry>
+    </visual>
+    <collision>
+      <origin xyz="0 0 0.1016358" rpy="0 0 0"/>
+      <geometry>
+        <mesh filename="package://marid_description/meshes/wheel.stl"/>
+      </geometry>
+    </collision>
+  </link>
+  <joint name="right_front_wheel_joint" type="continuous">
+    <parent link="right_front_wheel_arm"/>
+    <child link="right_front_wheel"/>
+    <origin xyz="0 0 -0.1016358" rpy="0 0 0"/>
+    <axis xyz="1 0 0"/>  <!-- Wheel rotation around own axle (parallel to world X) -->
+    <dynamics damping="0.01" friction="0.0"/>
+  </joint>
+  <link name="rear_wheel_arm">
+    <inertial>
+      <mass value="0.010886"/>
+      <origin xyz="0 0 -0.058191" rpy="0 0 0"/>  <!-- CoM from CAD (rear_arm), Z in m -->
+      <inertia ixx="6.145e-6" ixy="0" ixz="0" iyy="7.316e-6" iyz="0" izz="1.463e-6"/>  <!-- From CAD, kg⋅m² -->
+    </inertial>
+    <visual>
+      <origin xyz="0 0 0" rpy="0 0 0"/>
+      <geometry>
+        <mesh filename="package://marid_description/meshes/rear_wheel_arm.stl"/>
+      </geometry>
+    </visual>
+    <collision>
+      <origin xyz="0 0 0" rpy="0 0 0"/>
+      <geometry>
+        <mesh filename="package://marid_description/meshes/rear_wheel_arm.stl"/>
+      </geometry>
+    </collision>
+  </link>
+  <joint name="rear_arm_joint" type="fixed">
+    <parent link="base_link_front"/>
+    <child link="rear_wheel_arm"/>
+    <origin xyz="0 -0.28 -0.055" rpy="0 0 0"/>  <!-- Rear arm -->
+  </joint>
+  <link name="rear_wheel">
+    <inertial>
+      <mass value="0.05"/>  <!-- ~50 g, small landing wheel -->
+      <origin xyz="0 0 0" rpy="0 0 0"/>
+      <inertia ixx="7.8e-6" ixy="0" ixz="0" iyy="1.56e-5" iyz="0" izz="7.8e-6"/>  <!-- Disk r~0.025 m -->
+    </inertial>
+    <visual>
+      <origin xyz="0 0 0.1016358" rpy="0 0 0"/>
+      <geometry>
+        <mesh filename="package://marid_description/meshes/wheel.stl"/>
+      </geometry>
+    </visual>
+    <collision>
+      <origin xyz="0 0 0.1016358" rpy="0 0 0"/>
+      <geometry>
+        <mesh filename="package://marid_description/meshes/wheel.stl"/>
+      </geometry>
+    </collision>
+  </link>
+  <joint name="rear_wheel_joint" type="continuous">
+    <parent link="rear_wheel_arm"/>
+    <child link="rear_wheel"/>
+    <origin xyz="0 0 -0.1016358" rpy="0 0 0"/>
+    <axis xyz="1 0 0"/>  <!-- Wheel rotation around own axle (parallel to world X) -->
+    <dynamics damping="0.01" friction="0.0"/>
+  </joint>
   <link name="main_tail">
     <inertial>
@@ -327,45 +482,6 @@
       <mass value="0.05"/>
       <inertia ixx="1e-5" ixy="0" ixz="0" iyy="1e-5" iyz="0" izz="1e-5"/>
-      </inertial>
-      <!-- Hub/center cylinder -->
-      <visual>
-        <origin xyz="0 0 0" rpy="1.5708 0 0"/><geometry><cylinder length="0.1" radius="0.015"/></geometry>
-        <material name="red_thruster">
-          <color rgba="1.0 0.0 0.0 1.0"/>
-        </material>
-      </visual>
-      <!-- Propeller blade 1 - visible indicator for rotation -->
-      <visual>
-        <origin xyz="0.08 0 0" rpy="1.5708 0 0"/>
-        <geometry><box size="0.15 0.01 0.02"/></geometry>
-        <material name="red_thruster">
-          <color rgba="1.0 0.3 0.3 1.0"/>
-        </material>
-      </visual>
-      <!-- Propeller blade 2 - opposite side -->
-      <visual>
-        <origin xyz="-0.08 0 0" rpy="1.5708 0 0"/>
-        <geometry><box size="0.15 0.01 0.02"/></geometry>
-        <material name="red_thruster">
-          <color rgba="1.0 0.3 0.3 1.0"/>
-        </material>
-      </visual>
-      <!-- Propeller blade 3 - perpendicular -->
-      <visual>
-        <origin xyz="0 0.08 0" rpy="1.5708 0 0"/>
-        <geometry><box size="0.01 0.15 0.02"/></geometry>
-        <material name="red_thruster">
-          <color rgba="1.0 0.3 0.3 1.0"/>
-        </material>
-      </visual>
-      <!-- Propeller blade 4 - opposite -->
-      <visual>
-        <origin xyz="0 -0.08 0" rpy="1.5708 0 0"/>
-        <geometry><box size="0.01 0.15 0.02"/></geometry>
-        <material name="red_thruster">
-          <color rgba="1.0 0.3 0.3 1.0"/>
-        </material>
-      </visual>
-      <collision><origin xyz="0 0 0"/><geometry><cylinder length="0.1" radius="0.015"/></geometry></collision>
+    </inertial>
+    <collision><origin xyz="0 0 0"/><geometry><cylinder length="0.1" radius="0.015"/></geometry></collision>
   </link>
   <link name="thruster_R">
@@ -374,46 +490,6 @@
       <mass value="0.05"/>
       <inertia ixx="1e-5" ixy="0" ixz="0" iyy="1e-5" iyz="0" izz="1e-5"/>
-      </inertial>
-      <!-- Hub/center cylinder -->
-      <visual>
-        <origin xyz="0 0 0" rpy="1.5708 0 0"/>
-        <geometry><cylinder length="0.1" radius="0.015"/></geometry>
-        <material name="blue_thruster">
-          <color rgba="0.0 0.0 1.0 1.0"/>
-        </material>
-      </visual>
-      <!-- Propeller blade 1 - visible indicator for rotation -->
-      <visual>
-        <origin xyz="0.08 0 0" rpy="1.5708 0 0"/>
-        <geometry><box size="0.15 0.01 0.02"/></geometry>
-        <material name="blue_thruster">
-          <color rgba="0.3 0.3 1.0 1.0"/>
-        </material>
-      </visual>
-      <!-- Propeller blade 2 - opposite side -->
-      <visual>
-        <origin xyz="-0.08 0 0" rpy="1.5708 0 0"/>
-        <geometry><box size="0.15 0.01 0.02"/></geometry>
-        <material name="blue_thruster">
-          <color rgba="0.3 0.3 1.0 1.0"/>
-        </material>
-      </visual>
-      <!-- Propeller blade 3 - perpendicular -->
-      <visual>
-        <origin xyz="0 0.08 0" rpy="1.5708 0 0"/>
-        <geometry><box size="0.01 0.15 0.02"/></geometry>
-        <material name="blue_thruster">
-          <color rgba="0.3 0.3 1.0 1.0"/>
-        </material>
-      </visual>
-      <!-- Propeller blade 4 - opposite -->
-      <visual>
-        <origin xyz="0 -0.08 0" rpy="1.5708 0 0"/>
-        <geometry><box size="0.01 0.15 0.02"/></geometry>
-        <material name="blue_thruster">
-          <color rgba="0.3 0.3 1.0 1.0"/>
-        </material>
-      </visual>
-      <collision><origin xyz="0 0 0"/><geometry><cylinder length="0.1" radius="0.015"/></geometry></collision>
+    </inertial>
+    <collision><origin xyz="0 0 0"/><geometry><cylinder length="0.1" radius="0.015"/></geometry></collision>
   </link>
   <joint name="thruster_L_joint" type="continuous">

File: src/marid_description/urdf/marid_gazebo.xacro (robot description, xacro)
@@ -45,8 +45,8 @@
             <alpha_stall>0.35</alpha_stall>
             <forward>0 1 0</forward>
-            <up>0 0 1</up>
+            <upward>0 0 1</upward>
             <cp>0 0 0</cp>  <!-- Removed offset to prevent unwanted rotation -->
-            <debug>true</debug>  <!-- ADD DEBUG OUTPUT -->
-            <visualize>true</visualize>  <!-- VISUAL FORCES -->
+            <debug>true</debug>
+            <visualize>true</visualize>
         </plugin>
     </gazebo>
@@ -61,5 +61,5 @@
             <alpha_stall>0.35</alpha_stall>
             <forward>0 1 0</forward>
-            <up>0 0 1</up>
+            <upward>0 0 1</upward>
             <cp>0 0 0</cp>  <!-- Removed offset to prevent unwanted rotation -->
             <debug>true</debug>
@@ -77,8 +77,8 @@
             <alpha_stall>0.35</alpha_stall>
             <forward>0 1 0</forward>
-            <up>0 0 1</up>
+            <upward>0 0 1</upward>
             <cp>0 0 0</cp>  <!-- Removed offset to prevent unwanted rotation -->
-            <debug>true</debug>  <!-- ADD DEBUG OUTPUT -->
-            <visualize>true</visualize>  <!-- VISUAL FORCES -->
+            <debug>true</debug>
+            <visualize>true</visualize>
         </plugin>
     </gazebo>
@@ -93,5 +93,5 @@
             <alpha_stall>0.35</alpha_stall>
             <forward>0 1 0</forward>
-            <up>0 0 1</up>
+            <upward>0 0 1</upward>
             <cp>0 0 0</cp>  <!-- Removed offset to prevent unwanted rotation -->
             <debug>true</debug>
@@ -99,24 +99,9 @@
         </plugin>
     </gazebo>
-    <gazebo>
-        <plugin filename="libgz-sim8-lift-drag-system.so" name="gz::sim::systems::LiftDrag">
-            <link_name>base_link_front</link_name>
-            <air_density>1.225</air_density>  <!-- Air density at sea level (kg/m³) -->
-            <area>1.1425454568</area>
-            <a0>0.0</a0>  <!-- Zero-lift angle of attack (radians) -->
-            <cla>0.5</cla>  <!-- Added positive lift coefficient to counteract downward motion -->
-            <cda>0.2</cda>  <!-- Increased drag -->
-            <alpha_stall>1.57</alpha_stall>
-            <forward>0 1 0</forward>
-            <up>0 0 1</up>
-            <cp>0 0 0</cp>  <!-- No offset for fuselage -->
-            <debug>true</debug>
-        </plugin>
-    </gazebo>
     <!-- Aerodynamic Damping for Main Body (prevents uncontrolled rotations and drift) -->
-    <gazebo reference="base_link_front">
+    <gazebo reference="base_footprint">
         <plugin filename="libgz-sim8-hydrodynamics-system.so"
                 name="gz::sim::systems::Hydrodynamics">
-            <link_name>base_link_front</link_name>
+            <link_name>base_footprint</link_name>
             <!-- Linear drag coefficients (X, Y, Z) - acts like air resistance -->
             <xDotU>-0.5</xDotU>    <!-- Forward drag (X-axis) -->
@@ -153,7 +138,8 @@
             <alpha_stall>1.57</alpha_stall>
             <forward>0 1 0</forward>
-            <up>0 0 1</up>
+            <upward>0 0 1</upward>
             <cp>0 0 0</cp>  <!-- No offset for tail -->
             <debug>true</debug>
+            <visualize>true</visualize>
         </plugin>
     </gazebo>
