Commit message: Propulsion and aero: Thruster plugin, lift/drag, control surfaces, CG and mesh

File: src/marid_description/urdf/marid.urdf.xacro (robot description, xacro)
@@ -17,17 +17,9 @@
   <xacro:property name="right_wing_offset" value="0.0 ${-axis_offset_y} 0.0"/>
   <xacro:property name="wing_axis" value="1 0 0"/>
-  <!-- Spawn height: whole robot is lifted so it spawns above ground when model origin is at (0,0,0) -->
-  <xacro:property name="spawn_z_offset" value="0.12"/>
-  <!-- Root link at model origin (spawn point). No geometry/inertial needed. -->
-  <link name="base_footprint"/>
-  <joint name="base_footprint_joint" type="fixed">
-    <parent link="base_footprint"/>
-    <child link="base_link_front"/>
-    <origin xyz="0 0 ${spawn_z_offset}" rpy="0 0 0"/>
-  </joint>
+  <!-- Root link (spawn height set by launch file, e.g. -z 1.0) -->
   <link name="base_link_front">
     <inertial>
       <mass value="3.0903248"/>
-      <origin xyz="0 0.15 0" rpy="0 0 0"/>  <!-- COG moved forward to Y = 0.15 m to account for sensors, batteries, and electronics in front -->
+      <origin xyz="-2.54e-5 0.15 0" rpy="0 0 0"/>  <!-- COG: X from CAD (0.001 in right -> -2.54e-5 m here); Y = 0.15 m for sensors/batteries/electronics -->
       <inertia ixx="0.1110930358" ixy="0.0" ixz="0.0" iyy="0.0247075659" iyz="0.0" izz="0.1288539854"/>  <!-- Fixed: Zeroed iyz to eliminate cross-coupling moments -->
     </inertial>
@@ -117,5 +109,5 @@
     </collision>
   </link>
-  <joint name="left_front_wheel_joint" type="continuous">
+  <joint name="left_front_wheel_joint" type="fixed">
     <parent link="left_front_wheel_arm"/>
     <child link="left_front_wheel"/>
@@ -143,5 +135,5 @@
     </collision>
   </link>
-  <joint name="right_front_wheel_joint" type="continuous">
+  <joint name="right_front_wheel_joint" type="fixed">
     <parent link="right_front_wheel_arm"/>
     <child link="right_front_wheel"/>
@@ -193,5 +185,5 @@
     </collision>
   </link>
-  <joint name="rear_wheel_joint" type="continuous">
+  <joint name="rear_wheel_joint" type="fixed">
     <parent link="rear_wheel_arm"/>
     <child link="rear_wheel"/>
@@ -484,4 +476,11 @@
     </inertial>
     <collision><origin xyz="0 0 0"/><geometry><cylinder length="0.1" radius="0.015"/></geometry></collision>
+    <visual name="thruster_L_visual">
+      <origin xyz="0 0 0" rpy="0 0 0"/>
+      <geometry><cylinder length="0.1" radius="0.015"/></geometry>
+      <material name="red_thruster">
+        <color rgba="1.0 0.0 0.0 1.0"/>
+      </material>
+    </visual>
   </link>
   <link name="thruster_R">
@@ -492,4 +491,11 @@
     </inertial>
     <collision><origin xyz="0 0 0"/><geometry><cylinder length="0.1" radius="0.015"/></geometry></collision>
+    <visual name="thruster_R_visual">
+      <origin xyz="0 0 0" rpy="0 0 0"/>
+      <geometry><cylinder length="0.1" radius="0.015"/></geometry>
+      <material name="blue_thruster">
+        <color rgba="0.0 0.0 1.0 1.0"/>
+      </material>
+    </visual>
   </link>
   <joint name="thruster_L_joint" type="continuous">

File: src/marid_description/urdf/marid_gazebo.xacro (robot description, xacro)
@@ -35,146 +35,132 @@
         <maxVel>0.1</maxVel>
     </gazebo>
-    <gazebo>
-        <plugin filename="libgz-sim8-lift-drag-system.so" name="gz::sim::systems::LiftDrag">
-            <link_name>left_wing</link_name>
-            <air_density>1.225</air_density>  <!-- Air density at sea level (kg/m³) -->
-            <area>0.20674668328</area>  <!-- Increased for testing -->
-            <a0>0.0</a0>  <!-- Zero-lift angle of attack (radians) -->
-            <cla>3.0</cla>    <!-- Lift coefficient for wing -->
-            <cda>0.5</cda>     <!-- Increased drag -->
-            <alpha_stall>0.35</alpha_stall>
+    <!-- Aircraft-level aerodynamic model: AdvancedLiftDrag (single plugin) -->
+    <gazebo>
+        <plugin filename="gz-sim-advanced-lift-drag-system"
+                name="gz::sim::systems::AdvancedLiftDrag">
+            <!-- Coefficients copied from advanced_lift_drag demo as a starting point.
+                 These should be tuned for the MARID airframe. -->
+            <a0>0.0</a0>
+            <CL0>0.15188</CL0>
+            <AR>6.5</AR>
+            <eff>0.97</eff>
+            <CLa>5.015</CLa>
+            <CD0>0.029</CD0>
+            <Cem0>-0.075</Cem0>   <!-- Flipped for Y-forward: reduce nose-down tendency -->
+            <Cema>0.463966</Cema>
+            <CYb>-0.258244</CYb>
+            <Cellb>-0.03925</Cellb>
+            <Cenb>0.100826</Cenb>
+            <CDp>0.0</CDp>
+            <CYp>0.065861</CYp>
+            <CLp>0.0</CLp>
+            <Cellp>-0.487407</Cellp>
+            <Cemp>0.0</Cemp>
+            <Cenp>-0.040416</Cenp>
+            <CDq>0.055166</CDq>
+            <CYq>0.0</CYq>
+            <CLq>7.971792</CLq>
+            <Cellq>0.0</Cellq>
+            <Cemq>-12.14014</Cemq>
+            <Cenq>0.0</Cenq>
+            <CDr>0.0</CDr>
+            <CYr>0.230299</CYr>
+            <CLr>0.0</CLr>
+            <Cellr>0.078165</Cellr>
+            <Cemr>0.0</Cemr>
+            <Cenr>-0.089947</Cenr>
+            <alpha_stall>0.3391428111</alpha_stall>
+            <CLa_stall>-3.85</CLa_stall>
+            <CDa_stall>-0.9233984055</CDa_stall>
+            <Cema_stall>0</Cema_stall>
+            <!-- Aerodynamic reference geometry (approximate, to be tuned) -->
+            <cp>0 0 0</cp>          <!-- Aerodynamic center in base_link_front frame -->
+            <area>0.5</area>       <!-- Reference area (m²) for MARID aero model -->
+            <mac>0.22</mac>        <!-- Mean aerodynamic chord (m) -->
+            <air_density>1.225</air_density>
+            <!-- MARID coordinate convention: Y forward, Z up -->
             <forward>0 1 0</forward>
             <upward>0 0 1</upward>
-            <cp>0 0 0</cp>  <!-- Removed offset to prevent unwanted rotation -->
-            <debug>true</debug>
-            <visualize>true</visualize>
-        </plugin>
-    </gazebo>
-    <gazebo>
-        <plugin filename="libgz-sim8-lift-drag-system.so" name="gz::sim::systems::LiftDrag">
-            <link_name>right_wing</link_name>
-            <air_density>1.225</air_density>  <!-- Air density at sea level (kg/m³) -->
-            <area>0.20674668328</area>
-            <a0>0.0</a0>  <!-- Zero-lift angle of attack (radians) -->
-            <cla>3.0</cla>    <!-- Lift coefficient for wing -->
-            <cda>0.5</cda>
-            <alpha_stall>0.35</alpha_stall>
-            <forward>0 1 0</forward>
-            <upward>0 0 1</upward>
-            <cp>0 0 0</cp>  <!-- Removed offset to prevent unwanted rotation -->
-            <debug>true</debug>
-            <visualize>true</visualize>
-        </plugin>
-    </gazebo>
-    <gazebo>
-        <plugin filename="libgz-sim8-lift-drag-system.so" name="gz::sim::systems::LiftDrag">
-            <link_name>tail_left</link_name>
-            <air_density>1.225</air_density>  <!-- Air density at sea level (kg/m³) -->
-            <area>0.05733020792</area>  <!-- Increased for testing -->
-            <a0>0.0</a0>  <!-- Zero-lift angle of attack (radians) -->
-            <cla>0.8</cla>    <!-- Reasonable value for V-tail control surfaces -->
-            <cda>0.5</cda>     <!-- Increased drag -->
-            <alpha_stall>0.35</alpha_stall>
-            <forward>0 1 0</forward>
-            <upward>0 0 1</upward>
-            <cp>0 0 0</cp>  <!-- Removed offset to prevent unwanted rotation -->
-            <debug>true</debug>
-            <visualize>true</visualize>
-        </plugin>
-    </gazebo>
-    <gazebo>
-        <plugin filename="libgz-sim8-lift-drag-system.so" name="gz::sim::systems::LiftDrag">
-            <link_name>tail_right</link_name>
-            <air_density>1.225</air_density>  <!-- Air density at sea level (kg/m³) -->
-            <area>0.05733020792</area>
-            <a0>0.0</a0>  <!-- Zero-lift angle of attack (radians) -->
-            <cla>0.8</cla>    <!-- Reasonable value for V-tail control surfaces -->
-            <cda>0.5</cda>
-            <alpha_stall>0.35</alpha_stall>
-            <forward>0 1 0</forward>
-            <upward>0 0 1</upward>
-            <cp>0 0 0</cp>  <!-- Removed offset to prevent unwanted rotation -->
-            <debug>true</debug>
-            <visualize>true</visualize>
-        </plugin>
-    </gazebo>
-    <!-- Aerodynamic Damping for Main Body (prevents uncontrolled rotations and drift) -->
-    <gazebo reference="base_footprint">
-        <plugin filename="libgz-sim8-hydrodynamics-system.so"
-                name="gz::sim::systems::Hydrodynamics">
-            <link_name>base_footprint</link_name>
-            <!-- Linear drag coefficients (X, Y, Z) - acts like air resistance -->
-            <xDotU>-0.5</xDotU>    <!-- Forward drag (X-axis) -->
-            <yDotV>-1.0</yDotV>    <!-- Side drag (Y-axis - your forward) -->
-            <zDotW>-1.0</zDotW>    <!-- Vertical drag (Z-axis) -->
-            <!-- Angular drag coefficients (Roll, Pitch, Yaw) - rotational damping -->
-            <kDotP>-2.0</kDotP>    <!-- Roll damping (around X) -->
-            <mDotQ>-2.0</mDotQ>     <!-- Pitch damping (around Y) -->
-            <nDotR>-2.0</nDotR>     <!-- Yaw damping (around Z) -->
-            <!-- Quadratic drag (velocity-squared terms) -->
-            <xUabsU>-0.1</xUabsU>   <!-- Forward quadratic drag -->
-            <yVabsV>-0.2</yVabsV>   <!-- Side quadratic drag -->
-            <zWabsW>-0.2</zWabsW>   <!-- Vertical quadratic drag -->
-            <kPabsP>-1.0</kPabsP>  <!-- Roll quadratic damping -->
-            <mQabsQ>-1.0</mQabsQ>  <!-- Pitch quadratic damping -->
-            <nRabsR>-1.0</nRabsR>  <!-- Yaw quadratic damping -->
-            <!-- Linear velocity terms (usually zero for air) -->
-            <xU>0</xU>
-            <yV>0</yV>
-            <zW>0</zW>
-            <kP>0</kP>
-            <mQ>0</mQ>
-            <nR>0</nR>
-        </plugin>
-    </gazebo>
-    <gazebo reference="main_tail">
-        <plugin filename="libgz-sim8-lift-drag-system.so" name="gz::sim::systems::LiftDrag">
-            <link_name>main_tail</link_name>
-            <air_density>1.225</air_density>  <!-- Air density at sea level (kg/m³) -->
-            <area>0.1447926136</area>
-            <a0>0.0</a0>  <!-- Zero-lift angle of attack (radians) -->
-            <cla>0.4</cla>  <!-- Reverted to original value -->
-            <cda>0.15</cda>  <!-- Increased drag -->
-            <alpha_stall>1.57</alpha_stall>
-            <forward>0 1 0</forward>
-            <upward>0 0 1</upward>
-            <cp>0 0 0</cp>  <!-- No offset for tail -->
-            <debug>true</debug>
-            <visualize>true</visualize>
-        </plugin>
-    </gazebo>
-    <!-- ===== THRUSTER PLUGINS ===== -->
-    <!-- Left Thruster -->
-    <!-- Gazebo Sim 8 Thruster plugin uses default topic: /model/{namespace}/joint/{joint_name}/cmd_vel -->
+            <!-- Use the main fuselage link as the aero body -->
+            <link_name>base_link_front</link_name>
+            <!-- Control surfaces mapped to MARID joints (initial guess, to be tuned) -->
+            <num_ctrl_surfaces>4</num_ctrl_surfaces>
+            <!-- Left wing (aileron/elevon equivalent) -->
+            <control_surface>
+                <name>left_wing_joint</name>
+                <index>0</index>
+                <direction>-1</direction>   <!-- Match right wing: both wings -1 to fix right-side lift bias -->
+                <!-- Coefficients copied from reference servo_0 as a starting point -->
+                <CD_ctrl>-0.000059</CD_ctrl>
+                <CY_ctrl>0.000171</CY_ctrl>
+                <CL_ctrl>-0.011940</CL_ctrl>
+                <Cell_ctrl>-0.003331</Cell_ctrl>
+                <Cem_ctrl>0.001498</Cem_ctrl>
+                <Cen_ctrl>-0.000057</Cen_ctrl>
+            </control_surface>
+            <!-- Right wing; direction matches reference servo_1 -->
+            <control_surface>
+                <name>right_wing_joint</name>
+                <index>1</index>
+                <direction>1</direction>
+                <!-- From reference servo_1 -->
+                <CD_ctrl>-0.000059</CD_ctrl>
+                <CY_ctrl>-0.000171</CY_ctrl>
+                <CL_ctrl>-0.011940</CL_ctrl>
+                <Cell_ctrl>0.003331</Cell_ctrl>
+                <Cem_ctrl>0.001498</Cem_ctrl>
+                <Cen_ctrl>0.000057</Cen_ctrl>
+            </control_surface>
+            <!-- Left tail surface (V-tail); direction matches reference servo_2 -->
+            <control_surface>
+                <name>tail_left_joint</name>
+                <index>2</index>
+                <direction>-1</direction>
+                <!-- From reference servo_2 -->
+                <CD_ctrl>0.000274</CD_ctrl>
+                <CY_ctrl>0</CY_ctrl>
+                <CL_ctrl>0.010696</CL_ctrl>
+                <Cell_ctrl>0.0</Cell_ctrl>
+                <Cem_ctrl>-0.025798</Cem_ctrl>
+                <Cen_ctrl>0.0</Cen_ctrl>
+            </control_surface>
+            <!-- Right tail surface (V-tail); direction matches reference servo_3 -->
+            <control_surface>
+                <name>tail_right_joint</name>
+                <index>3</index>
+                <direction>1</direction>
+                <!-- From reference servo_3 -->
+                <CD_ctrl>0.0</CD_ctrl>
+                <CY_ctrl>-0.003913</CY_ctrl>
+                <CL_ctrl>0.0</CL_ctrl>
+                <Cell_ctrl>-0.000257</Cell_ctrl>
+                <Cem_ctrl>0.0</Cem_ctrl>
+                <Cen_ctrl>0.001613</Cen_ctrl>
+            </control_surface>
+        </plugin>
+    </gazebo>
+    <!-- ===== THRUSTER PLUGIN (force in Newtons, no reaction torque on body) ===== -->
+    <!-- Center: topic /model/marid/joint/thruster_center_joint/cmd_thrust (gz.msgs.Double, force N) -->
     <gazebo>
         <plugin filename="libgz-sim8-thruster-system.so" name="gz::sim::systems::Thruster">
-            <namespace>marid</namespace>
+            <joint_name>thruster_center_joint</joint_name>
+            <fluid_density>1.204</fluid_density>
+            <propeller_diameter>0.03</propeller_diameter>
+        </plugin>
+    </gazebo>
+    <!-- Left: topic /model/marid/joint/thruster_L_joint/cmd_thrust -->
+    <gazebo>
+        <plugin filename="libgz-sim8-thruster-system.so" name="gz::sim::systems::Thruster">
             <joint_name>thruster_L_joint</joint_name>
-            <fluid_density>1.225</fluid_density>  <!-- Air density at sea level (kg/m³) -->
-            <propeller_diameter>0.2</propeller_diameter>  <!-- Adjust based on your propeller size (meters) -->
-            <thrust_coefficient>0.8</thrust_coefficient>  <!-- Typical range: 0.6-1.0 -->
-            <use_angvel_cmd>true</use_angvel_cmd>  <!-- Accept angular velocity commands (rad/s) -->
-        </plugin>
-    </gazebo>
-    <!-- Right Thruster -->
+            <fluid_density>1.204</fluid_density>
+            <propeller_diameter>0.03</propeller_diameter>
+        </plugin>
+    </gazebo>
+    <!-- Right: topic /model/marid/joint/thruster_R_joint/cmd_thrust -->
     <gazebo>
         <plugin filename="libgz-sim8-thruster-system.so" name="gz::sim::systems::Thruster">
-            <namespace>marid</namespace>
             <joint_name>thruster_R_joint</joint_name>
-            <fluid_density>1.225</fluid_density>
-            <propeller_diameter>0.2</propeller_diameter>
-            <thrust_coefficient>0.8</thrust_coefficient>  <!-- Typical range: 0.6-1.0 -->
-            <use_angvel_cmd>true</use_angvel_cmd>
-        </plugin>
-    </gazebo>
-    <!-- Center Thruster (for single-thruster testing) -->
-    <gazebo>
-        <plugin filename="libgz-sim8-thruster-system.so" name="gz::sim::systems::Thruster">
-            <namespace>marid</namespace>
-            <joint_name>thruster_center_joint</joint_name>
-            <fluid_density>1.225</fluid_density>
-            <propeller_diameter>0.2</propeller_diameter>
-            <thrust_coefficient>0.8</thrust_coefficient>
-            <use_angvel_cmd>true</use_angvel_cmd>
+            <fluid_density>1.204</fluid_density>
+            <propeller_diameter>0.03</propeller_diameter>
         </plugin>
     </gazebo>
