Commit message: Add MARID new design: larger scale, closer to real vehicle; fix URDF and refs
Introduce a second MARID model variant (marid_new) for the updated design:
- New URDF (marid_new.urdf.xacro), Gazebo plugins (marid_new_gazebo.xacro),
  and launch files (gazebo_new, display_new) for the new design.
- Larger scale and geometry closer to the real vehicle; X-forward convention;
  meshes in meshes_2/; tuned mass/inertia and aero (AdvancedLiftDrag,
  Hydrodynamics) for the bigger airframe.
- Thruster plugins: increased thrust limits (max_thrust_cmd/min_thrust_cmd)
  and propeller diameter for the main thruster; wheel joints optionally fixed
  for testing.
- URDF: remove invalid axis/limit from fixed joints; correct thruster and
  nose-prop comments for X-forward; align GPS/LIDAR/pitot comments with
  origins; remove redundant IMU joint axis.
- Gazebo: fix rear wheel plugin reference (left_rear_wheel -> rear_wheel);
  clarify thruster coefficient comment.
- Launch: bridge uses /world/empty/state to match default world; add note
  when using another world.

File: src/marid_description/urdf/marid_new.urdf.xacro (robot description, xacro)
@@ -3,5 +3,5 @@
   <xacro:arg name="is_ignition" default="true"/>
   <!-- Include Gazebo parameters-->
-  <xacro:include filename="$(find marid_description)/urdf/marid_gazebo.xacro"/>
+  <xacro:include filename="$(find marid_description)/urdf/marid_new_gazebo.xacro"/>
   <!-- ROS2 Control Library-->
   <xacro:include filename="$(find marid_description)/urdf/marid_ros2_control.xacro"/>
@@ -20,18 +20,21 @@
   <link name="base_link_front">
     <inertial>
-      <mass value="3.0903248"/>
-      <origin xyz="0 0 0" rpy="0 0 1.5708"/>  <!-- COG: symmetric CAD (X=0); Y = 0.15 m for sensors/batteries/electronics -->
-      <inertia ixx="0.1110930358" ixy="0.0" ixz="0.0" iyy="0.0247075659" iyz="0.0" izz="0.1288539854"/>  <!-- Fixed: Zeroed iyz to eliminate cross-coupling moments -->
-    </inertial>
-    <visual>
-      <origin xyz="0 0 0" rpy="0 0 0"/>
-      <geometry>
-        <mesh filename="package://marid_description/meshes/base_link_front.stl"/>
-      </geometry>
-    </visual>
-    <collision>
-      <origin xyz="0 0 0" rpy="0 0 0"/>
-      <geometry>
-        <box size="0.25 0.45 0.12"/>
+      <mass value="84.735"/>
+      <origin xyz="-1.876 0 0.306" rpy="0 0 0"/>  <!-- COG already placed correctly -->
+      <inertia ixx="6.643" ixy="0.013" ixz="-0.151" iyy="49.838" iyz="0.001" izz="55.184"/>
+    </inertial>
+    <visual>
+      <origin xyz="0 0 0" rpy="0 0 0"/>
+      <geometry>
+        <mesh filename="package://marid_description/meshes_2/base_link_front.stl"/>
+      </geometry>
+      <material name="base_link_front_dark_grey">
+        <color rgba="0.2 0.2 0.2 1.0"/>
+      </material>
+    </visual>
+    <collision>
+      <origin xyz="0 0 0" rpy="0 0 0"/>
+      <geometry>
+        <mesh filename="package://marid_description/meshes_2/base_link_front.stl"/>
       </geometry>
     </collision>
@@ -40,18 +43,21 @@
   <link name="left_front_wheel_arm">
     <inertial>
-      <mass value="0.005443"/>
-      <origin xyz="0 0 -0.069215" rpy="0 0 0"/>  <!-- CoM from CAD (front_wheel_arm), Z in m -->
-      <inertia ixx="1.756e-6" ixy="0" ixz="0" iyy="2.048e-6" iyz="0" izz="2.926e-7"/>  <!-- From CAD, kg⋅m² -->
-    </inertial>
-    <visual>
-      <origin xyz="0 0 0" rpy="0 0 0"/>
-      <geometry>
-        <mesh filename="package://marid_description/meshes/front_wheel_arm.stl"/>
-      </geometry>
-    </visual>
-    <collision>
-      <origin xyz="0 0 0" rpy="0 0 0"/>
-      <geometry>
-        <mesh filename="package://marid_description/meshes/front_wheel_arm.stl"/>
+      <mass value="0.392"/>
+      <origin xyz="-0.525 0.20786886 -0.00022077" rpy="0 0 0"/>
+      <inertia ixx="0.002" ixy="0.0" ixz="0.0" iyy="0.002" iyz="0.0" izz="3.794e-4"/>
+    </inertial>
+    <visual>
+      <origin xyz="0 0 0" rpy="0 0 0"/>
+      <geometry>
+        <mesh filename="package://marid_description/meshes_2/front_left_arm.stl"/>
+      </geometry>
+      <material name="arm_black">
+        <color rgba="0.1 0.1 0.1 1.0"/>
+      </material>
+    </visual>
+    <collision>
+      <origin xyz="0 0 0" rpy="0 0 0"/>
+      <geometry>
+        <mesh filename="package://marid_description/meshes_2/front_left_arm.stl"/>
       </geometry>
     </collision>
@@ -60,24 +66,25 @@
     <parent link="base_link_front"/>
     <child link="left_front_wheel_arm"/>
-    <origin xyz="-0.053 0.355 -0.069" rpy="0 0 0"/>  <!-- Top of left arm from CAD (min dist), m; Z neg = below origin -->
-    <axis xyz="0 1 0"/>
-    <limit lower="0" upper="0" effort="1000" velocity="1000"/>
+    <origin xyz="0 0 0" rpy="0 0 0"/>  <!-- Top of left arm from CAD (min dist), m; Z neg = below origin -->
   </joint>
   <link name="right_front_wheel_arm">
     <inertial>
-      <mass value="0.005443"/>
-      <origin xyz="0 0 -0.069215" rpy="0 0 0"/>  <!-- CoM from CAD (front_wheel_arm), Z in m -->
-      <inertia ixx="1.756e-6" ixy="0" ixz="0" iyy="2.048e-6" iyz="0" izz="2.926e-7"/>  <!-- From CAD, kg⋅m² -->
-    </inertial>
-    <visual>
-      <origin xyz="0 0 0" rpy="0 0 0"/>
-      <geometry>
-        <mesh filename="package://marid_description/meshes/front_wheel_arm.stl"/>
-      </geometry>
-    </visual>
-    <collision>
-      <origin xyz="0 0 0" rpy="0 0 0"/>
-      <geometry>
-        <mesh filename="package://marid_description/meshes/front_wheel_arm.stl"/>
+      <mass value="0.392"/>
+      <origin xyz="-0.525 -0.20786886 -0.00022077" rpy="0 0 0"/>
+      <inertia ixx="0.002" ixy="0.0" ixz="0.0" iyy="0.002" iyz="0.0" izz="3.794e-4"/>
+    </inertial>
+    <visual>
+      <origin xyz="0 0 0" rpy="0 0 0"/>
+      <geometry>
+        <mesh filename="package://marid_description/meshes_2/front_right_arm.stl"/>
+      </geometry>
+      <material name="arm_black">
+        <color rgba="0.1 0.1 0.1 1.0"/>
+      </material>
+    </visual>
+    <collision>
+      <origin xyz="0 0 0" rpy="0 0 0"/>
+      <geometry>
+        <mesh filename="package://marid_description/meshes_2/front_right_arm.stl"/>
       </geometry>
     </collision>
@@ -86,76 +93,79 @@
     <parent link="base_link_front"/>
     <child link="right_front_wheel_arm"/>
-    <origin xyz="0.053 0.355 -0.069" rpy="0 0 0"/>  <!-- Top of right arm from CAD (min dist), m; Z neg = below origin -->
-    <axis xyz="0 1 0"/>
-    <limit lower="0" upper="0" effort="1000" velocity="1000"/>
+    <origin xyz="0 0 0" rpy="0 0 0"/>  <!-- Top of right arm from CAD (min dist), m; Z neg = below origin -->
   </joint>
   <link name="left_front_wheel">
     <inertial>
-      <mass value="0.05"/>  <!-- ~50 g, small landing wheel -->
-      <origin xyz="0 0 0" rpy="0 0 0"/>
-      <inertia ixx="7.8e-6" ixy="0" ixz="0" iyy="1.56e-5" iyz="0" izz="7.8e-6"/>  <!-- Disk r~0.025 m: I_ax=0.5*m*r^2, I_rad=0.25*m*r^2 -->
-    </inertial>
-    <visual>
-      <origin xyz="0 0 0.1016358" rpy="0 0 0"/>
-      <geometry>
-        <mesh filename="package://marid_description/meshes/wheel.stl"/>
-      </geometry>
-    </visual>
-    <collision>
-      <origin xyz="0 0 0.1016358" rpy="0 0 0"/>
-      <geometry>
-        <mesh filename="package://marid_description/meshes/wheel.stl"/>
-      </geometry>
-    </collision>
-  </link>
-  <joint name="left_front_wheel_joint" type="fixed">
+      <mass value="0.934"/>
+      <origin xyz="0.525 -0.20786886 0.09000082" rpy="0 0 0"/>
+      <inertia ixx="0.0036" ixy="0" ixz="0" iyy="0.007" iyz="0" izz="0.0036"/>
+    </inertial>
+    <visual>
+      <origin xyz="0.525 -0.20786886 0.09000082" rpy="0 0 0"/>
+      <geometry>
+        <mesh filename="package://marid_description/meshes_2/front_left_tire.stl"/>
+      </geometry>
+      <material name="tire_black">
+        <color rgba="0.1 0.1 0.1 1.0"/>
+      </material>
+    </visual>
+    <collision>
+      <origin xyz="0.525 -0.20786886 0.09000082" rpy="0 0 0"/>
+      <geometry>
+        <mesh filename="package://marid_description/meshes_2/front_left_tire.stl"/>
+      </geometry>
+    </collision>
+  </link>
+  <joint name="left_front_wheel_joint" type="fixed">  <!-- fixed for testing (was continuous) -->
     <parent link="left_front_wheel_arm"/>
     <child link="left_front_wheel"/>
-    <origin xyz="0 0 -0.1016358" rpy="0 0 0"/>
-    <axis xyz="1 0 0"/>  <!-- Wheel rotation around own axle (parallel to world X) -->
-    <dynamics damping="0.01" friction="0.0"/>
+    <origin xyz="-0.525 0.20786886 -0.09000082" rpy="0 0 0"/>
   </joint>
   <link name="right_front_wheel">
     <inertial>
-      <mass value="0.05"/>  <!-- ~50 g, small landing wheel -->
-      <origin xyz="0 0 0" rpy="0 0 0"/>
-      <inertia ixx="7.8e-6" ixy="0" ixz="0" iyy="1.56e-5" iyz="0" izz="7.8e-6"/>  <!-- Disk r~0.025 m: I_ax=0.5*m*r^2, I_rad=0.25*m*r^2 -->
-    </inertial>
-    <visual>
-      <origin xyz="0 0 0.1016358" rpy="0 0 0"/>
-      <geometry>
-        <mesh filename="package://marid_description/meshes/wheel.stl"/>
-      </geometry>
-    </visual>
-    <collision>
-      <origin xyz="0 0 0.1016358" rpy="0 0 0"/>
-      <geometry>
-        <mesh filename="package://marid_description/meshes/wheel.stl"/>
-      </geometry>
-    </collision>
-  </link>
-  <joint name="right_front_wheel_joint" type="fixed">
+      <mass value="0.934"/>
+      <origin xyz="0.525 0.20786886 0.09000082" rpy="0 0 0"/>
+      <inertia ixx="0.0036" ixy="0" ixz="0" iyy="0.007" iyz="0" izz="0.0036"/>
+    </inertial>
+    <visual>
+      <origin xyz="0.525 0.20786886 0.09000082" rpy="0 0 0"/>
+      <geometry>
+        <mesh filename="package://marid_description/meshes_2/front_right_tire.stl"/>
+      </geometry>
+      <material name="tire_black">
+        <color rgba="0.1 0.1 0.1 1.0"/>
+      </material>
+    </visual>
+    <collision>
+      <origin xyz="0.525 0.20786886 0.09000082" rpy="0 0 0"/>
+      <geometry>
+        <mesh filename="package://marid_description/meshes_2/front_right_tire.stl"/>
+      </geometry>
+    </collision>
+  </link>
+  <joint name="right_front_wheel_joint" type="fixed">  <!-- fixed for testing (was continuous) -->
     <parent link="right_front_wheel_arm"/>
     <child link="right_front_wheel"/>
-    <origin xyz="0 0 -0.1016358" rpy="0 0 0"/>
-    <axis xyz="1 0 0"/>  <!-- Wheel rotation around own axle (parallel to world X) -->
-    <dynamics damping="0.01" friction="0.0"/>
+    <origin xyz="-0.525 -0.20786886 -0.09000082" rpy="0 0 0"/>
   </joint>
   <link name="rear_wheel_arm">
     <inertial>
-      <mass value="0.010886"/>
-      <origin xyz="0 0 -0.058191" rpy="0 0 0"/>  <!-- CoM from CAD (rear_arm), Z in m -->
-      <inertia ixx="6.145e-6" ixy="0" ixz="0" iyy="7.316e-6" iyz="0" izz="1.463e-6"/>  <!-- From CAD, kg⋅m² -->
-    </inertial>
-    <visual>
-      <origin xyz="0 0 0" rpy="0 0 0"/>
-      <geometry>
-        <mesh filename="package://marid_description/meshes/rear_wheel_arm.stl"/>
-      </geometry>
-    </visual>
-    <collision>
-      <origin xyz="0 0 0" rpy="0 0 0"/>
-      <geometry>
-        <mesh filename="package://marid_description/meshes/rear_wheel_arm.stl"/>
+      <mass value="0.362"/>
+      <origin xyz="-2.47499035 0 0.05355912" rpy="0 0 0"/>
+      <inertia ixx="0.001" ixy="0.0" ixz="-3.417e-7" iyy="0.001" iyz="0.0" izz="3.242e-4"/>
+    </inertial>
+    <visual>
+      <origin xyz="0 0 0" rpy="0 0 0"/>
+      <geometry>
+        <mesh filename="package://marid_description/meshes_2/rear_arm.stl"/>
+      </geometry>
+      <material name="arm_black">
+        <color rgba="0.1 0.1 0.1 1.0"/>
+      </material>
+    </visual>
+    <collision>
+      <origin xyz="0 0 0" rpy="0 0 0"/>
+      <geometry>
+        <mesh filename="package://marid_description/meshes_2/rear_arm.stl"/>
       </geometry>
     </collision>
@@ -164,48 +174,52 @@
     <parent link="base_link_front"/>
     <child link="rear_wheel_arm"/>
-    <origin xyz="0 -0.28 -0.055" rpy="0 0 0"/>  <!-- Rear arm -->
+    <origin xyz="0 0 0" rpy="0 0 0"/>  <!-- Rear arm -->
   </joint>
   <link name="rear_wheel">
     <inertial>
-      <mass value="0.05"/>  <!-- ~50 g, small landing wheel -->
-      <origin xyz="0 0 0" rpy="0 0 0"/>
-      <inertia ixx="7.8e-6" ixy="0" ixz="0" iyy="1.56e-5" iyz="0" izz="7.8e-6"/>  <!-- Disk r~0.025 m -->
-    </inertial>
-    <visual>
-      <origin xyz="0 0 0.1016358" rpy="0 0 0"/>
-      <geometry>
-        <mesh filename="package://marid_description/meshes/wheel.stl"/>
-      </geometry>
-    </visual>
-    <collision>
-      <origin xyz="0 0 0.1016358" rpy="0 0 0"/>
-      <geometry>
-        <mesh filename="package://marid_description/meshes/wheel.stl"/>
-      </geometry>
-    </collision>
-  </link>
-  <joint name="rear_wheel_joint" type="fixed">
+      <mass value="0.573"/>
+      <origin xyz="2.475 0 0.02500082" rpy="0 0 0"/>
+      <inertia ixx="0.0016" ixy="0" ixz="0" iyy="0.003" iyz="0" izz="0.0016"/>
+    </inertial>
+    <visual>
+      <origin xyz="2.475 0 0.02500082" rpy="0 0 0"/>
+      <geometry>
+        <mesh filename="package://marid_description/meshes_2/rear_tire.stl"/>
+      </geometry>
+      <material name="tire_black">
+        <color rgba="0.1 0.1 0.1 1.0"/>
+      </material>
+    </visual>
+    <collision>
+      <origin xyz="2.475 0 0.02500082" rpy="0 0 0"/>
+      <geometry>
+        <mesh filename="package://marid_description/meshes_2/rear_tire.stl"/>
+      </geometry>
+    </collision>
+  </link>
+  <joint name="rear_wheel_joint" type="fixed">  <!-- fixed for testing (was continuous) -->
     <parent link="rear_wheel_arm"/>
     <child link="rear_wheel"/>
-    <origin xyz="0 0 -0.1016358" rpy="0 0 0"/>
-    <axis xyz="1 0 0"/>  <!-- Wheel rotation around own axle (parallel to world X) -->
-    <dynamics damping="0.01" friction="0.0"/>
+    <origin xyz="-2.475 0 -0.02500082" rpy="0 0 0"/>
   </joint>
   <link name="main_tail">
     <inertial>
-      <mass value="0.69082118"/>
-      <origin xyz="0 0.1 0.02" rpy="0 0 0"/>
-      <inertia ixx="0.0077116401" ixy="0.0" ixz="0.0" iyy="0.0006628288" iyz="0.0" izz="0.0077111242"/>
-    </inertial>
-    <visual>
-      <origin xyz="0 0 0" rpy="0 0 0"/>
-      <geometry>
-        <mesh filename="package://marid_description/meshes/main_tail.stl"/>
-      </geometry>
-    </visual>
-    <collision>
-      <origin xyz="0 0 0" rpy="0 0 0"/>
-      <geometry>
-        <box size="0.15 0.25 0.06"/>
+      <mass value="17.551"/>
+      <origin xyz="-2.4135434 0 0.34612528" rpy="0 0 0"/>
+      <inertia ixx="1.073" ixy="1.867e-6" ixz="-0.023" iyy="2.113" iyz="-2.847e-7" izz="3.168"/>
+    </inertial>
+    <visual>
+      <origin xyz="0 0 0" rpy="0 0 0"/>
+      <geometry>
+        <mesh filename="package://marid_description/meshes_2/main_tail.stl"/>
+      </geometry>
+      <material name="main_tail_black">
+        <color rgba="0.1 0.1 0.1 1.0"/>
+      </material>
+    </visual>
+    <collision>
+      <origin xyz="0 0 0" rpy="0 0 0"/>
+      <geometry>
+        <mesh filename="package://marid_description/meshes_2/main_tail.stl"/>
       </geometry>
     </collision>
@@ -214,36 +228,34 @@
     <parent link="base_link_front"/>
     <child link="main_tail"/>
-    <origin xyz="0 -.2115 -0.0555" rpy="0 0 0"/>
+    <origin xyz="0 0 0" rpy="0 0 0"/>
+  </joint>
+  <link name="left_wing">
+    <inertial>
+      <origin xyz="-1.72531399 1.11004875 0.18389363" rpy="0 0 0"/>
+      <mass value="3.662"/>
+      <inertia ixx="0.55" ixy="0.54" ixz="-0.022" iyy="0.662" iyz="0.021" izz="1.202"/>
+    </inertial>
+    <visual>
+      <origin xyz="1.225 -0.5 -0.208" rpy="0 0 0"/>
+      <geometry>
+        <mesh filename="package://marid_description/meshes_2/left_wing.stl"/>
+      </geometry>
+      <material name="wing_black">
+        <color rgba="0.1 0.1 0.1 1.0"/>
+      </material>
+    </visual>
+    <collision>
+      <origin xyz="1.225 -0.5 -0.208" rpy="0 0 0"/>
+      <geometry>
+        <mesh filename="package://marid_description/meshes_2/left_wing.stl"/>
+      </geometry>
+    </collision>
+  </link>
+  <joint name="left_wing_joint" type="revolute">
+    <parent link="base_link_front"/>
+    <child link="left_wing"/>
+    <origin xyz="-1.225 0.5 0.208" rpy="0 0 0"/>
     <axis xyz="0 1 0"/>
-    <limit lower="0" upper="0" effort="1000" velocity="1000"/>
-  </joint>
-  <link name="left_wing">
-    <inertial>
-      <origin xyz="${left_wing_offset}" rpy="0 0 0"/>
-      <mass value="1.44"/>
-      <inertia ixx="0.0139618379" ixy="-0.0200668863" ixz="0.003481534" iyy="0.0399031726" iyz="0.001971806" izz="0.0531650164"/>
-    </inertial>
-    <visual>
-      <origin xyz="${left_wing_offset}" rpy="0 0 0"/>
-      <geometry>
-        <mesh filename="package://marid_description/meshes/left_wing.stl"/>
-      </geometry>
-      <material name="left_wing_red">
-        <color rgba="1.0 0.0 0.0 1.0"/>
-      </material>
-    </visual>
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