Commit message: Tune MARID new model inertials and aero for stable flight
- Recomputed inertial origins for wings, tails, wheels and thrusters in marid_new.urdf.xacro
  so CoMs live in their own link frames instead of at joint origins.
- Tuned V-tail joint axes, inertial offsets, and AdvancedLiftDrag control-surface
  coefficients (Cem/Cen, direction) so symmetric deflection gives mostly pitch and
  differential deflection gives yaw, matching the reference advanced_lift_drag demo.
- Updated Hydrodynamics damping for base_link_front (linear and quadratic terms) to
  provide strong but reasonable aero damping for the larger, heavier airframe.
- Adjusted wing and tail joint dynamics (friction/effort) and joint position controller
  p_gains so control surfaces resist gravity and aero loads but remain responsive
  only to commanded deflections.

File: src/marid_description/urdf/marid_new.urdf.xacro (robot description, xacro)
@@ -6,16 +6,10 @@
   <!-- ROS2 Control Library-->
   <xacro:include filename="$(find marid_description)/urdf/marid_ros2_control.xacro"/>
-  <!-- Axis translation along y - adjust this value as needed -->
-  <xacro:property name="axis_offset_y" value="0.1"/>
-  <!-- Joint origins at the desired rotation axis location -->
-  <xacro:property name="left_wing_xyz" value="0.0 ${0.18 + axis_offset_y} -0.04"/>
-  <xacro:property name="left_wing_rpy" value="0.0 0.0 0.0"/>
-  <xacro:property name="right_wing_xyz" value="0.0 ${0.18 + axis_offset_y} -0.04"/>
-  <xacro:property name="right_wing_rpy" value="0.0 0.0 0.0"/>
-  <!-- Offset for wing geometry relative to joint (to keep wing in original position) -->
-  <xacro:property name="left_wing_offset" value="0.0 ${-axis_offset_y} 0.0"/>
-  <xacro:property name="right_wing_offset" value="0.0 ${-axis_offset_y} 0.0"/>
-  <xacro:property name="wing_axis" value="1 0 0"/>
-  <!-- Root link (spawn height set by launch file, e.g. -z 1.0) -->
+  <!-- Joint origins at the desired rotation axis location; inertial origin = CoM in link frame (computed from joint origin) -->
+  <xacro:property name="left_wing_inertial" value="-0.50031399 0.61004875 -0.02410637"/>
+  <xacro:property name="right_wing_inertial" value="-0.50031399 -0.61004875 -0.02410637"/>
+  <!-- Tail V-surfaces: inertial origin = CoM in tail link frame.-->
+  <xacro:property name="tail_left_inertial" value="-0.12167064 0.13072223 0.12984906"/>
+  <xacro:property name="tail_right_inertial" value="-0.12167064 -0.13072223 0.12984906"/>
   <link name="base_link_front">
     <inertial>
@@ -98,24 +92,24 @@
     <inertial>
       <mass value="0.934"/>
+      <origin xyz="0 0 0" rpy="0 0 0"/>
+      <inertia ixx="0.0036" ixy="0" ixz="0" iyy="0.007" iyz="0" izz="0.0036"/>
+    </inertial>
+    <visual>
       <origin xyz="0.525 -0.20786886 0.09000082" rpy="0 0 0"/>
-      <inertia ixx="0.0036" ixy="0" ixz="0" iyy="0.007" iyz="0" izz="0.0036"/>
-    </inertial>
-    <visual>
+      <geometry>
+        <mesh filename="package://marid_description/meshes_2/front_left_tire.stl"/>
+      </geometry>
+      <material name="tire_black">
+        <color rgba="0.1 0.1 0.1 1.0"/>
+      </material>
+    </visual>
+    <collision>
       <origin xyz="0.525 -0.20786886 0.09000082" rpy="0 0 0"/>
       <geometry>
         <mesh filename="package://marid_description/meshes_2/front_left_tire.stl"/>
       </geometry>
-      <material name="tire_black">
-        <color rgba="0.1 0.1 0.1 1.0"/>
-      </material>
-    </visual>
-    <collision>
-      <origin xyz="0.525 -0.20786886 0.09000082" rpy="0 0 0"/>
-      <geometry>
-        <mesh filename="package://marid_description/meshes_2/front_left_tire.stl"/>
-      </geometry>
-    </collision>
-  </link>
-  <joint name="left_front_wheel_joint" type="fixed">  <!-- fixed for testing (was continuous) -->
+    </collision>
+  </link>
+  <joint name="left_front_wheel_joint" type="fixed">
     <parent link="left_front_wheel_arm"/>
     <child link="left_front_wheel"/>
@@ -125,24 +119,24 @@
     <inertial>
       <mass value="0.934"/>
+      <origin xyz="0 0 0" rpy="0 0 0"/>
+      <inertia ixx="0.0036" ixy="0" ixz="0" iyy="0.007" iyz="0" izz="0.0036"/>
+    </inertial>
+    <visual>
       <origin xyz="0.525 0.20786886 0.09000082" rpy="0 0 0"/>
-      <inertia ixx="0.0036" ixy="0" ixz="0" iyy="0.007" iyz="0" izz="0.0036"/>
-    </inertial>
-    <visual>
+      <geometry>
+        <mesh filename="package://marid_description/meshes_2/front_right_tire.stl"/>
+      </geometry>
+      <material name="tire_black">
+        <color rgba="0.1 0.1 0.1 1.0"/>
+      </material>
+    </visual>
+    <collision>
       <origin xyz="0.525 0.20786886 0.09000082" rpy="0 0 0"/>
       <geometry>
         <mesh filename="package://marid_description/meshes_2/front_right_tire.stl"/>
       </geometry>
-      <material name="tire_black">
-        <color rgba="0.1 0.1 0.1 1.0"/>
-      </material>
-    </visual>
-    <collision>
-      <origin xyz="0.525 0.20786886 0.09000082" rpy="0 0 0"/>
-      <geometry>
-        <mesh filename="package://marid_description/meshes_2/front_right_tire.stl"/>
-      </geometry>
-    </collision>
-  </link>
-  <joint name="right_front_wheel_joint" type="fixed">  <!-- fixed for testing (was continuous) -->
+    </collision>
+  </link>
+  <joint name="right_front_wheel_joint" type="fixed">
     <parent link="right_front_wheel_arm"/>
     <child link="right_front_wheel"/>
@@ -179,24 +173,24 @@
     <inertial>
       <mass value="0.573"/>
+      <origin xyz="0 0 0" rpy="0 0 0"/>
+      <inertia ixx="0.0016" ixy="0" ixz="0" iyy="0.003" iyz="0" izz="0.0016"/>
+    </inertial>
+    <visual>
       <origin xyz="2.475 0 0.02500082" rpy="0 0 0"/>
-      <inertia ixx="0.0016" ixy="0" ixz="0" iyy="0.003" iyz="0" izz="0.0016"/>
-    </inertial>
-    <visual>
+      <geometry>
+        <mesh filename="package://marid_description/meshes_2/rear_tire.stl"/>
+      </geometry>
+      <material name="tire_black">
+        <color rgba="0.1 0.1 0.1 1.0"/>
+      </material>
+    </visual>
+    <collision>
       <origin xyz="2.475 0 0.02500082" rpy="0 0 0"/>
       <geometry>
         <mesh filename="package://marid_description/meshes_2/rear_tire.stl"/>
       </geometry>
-      <material name="tire_black">
-        <color rgba="0.1 0.1 0.1 1.0"/>
-      </material>
-    </visual>
-    <collision>
-      <origin xyz="2.475 0 0.02500082" rpy="0 0 0"/>
-      <geometry>
-        <mesh filename="package://marid_description/meshes_2/rear_tire.stl"/>
-      </geometry>
-    </collision>
-  </link>
-  <joint name="rear_wheel_joint" type="fixed">  <!-- fixed for testing (was continuous) -->
+    </collision>
+  </link>
+  <joint name="rear_wheel_joint" type="fixed">
     <parent link="rear_wheel_arm"/>
     <child link="rear_wheel"/>
@@ -232,5 +226,5 @@
   <link name="left_wing">
     <inertial>
-      <origin xyz="-1.72531399 1.11004875 0.18389363" rpy="0 0 0"/>
+      <origin xyz="${left_wing_inertial}" rpy="0 0 0"/>
       <mass value="3.662"/>
       <inertia ixx="0.55" ixy="0.54" ixz="-0.022" iyy="0.662" iyz="0.021" izz="1.202"/>
@@ -257,5 +251,5 @@
     <origin xyz="-1.225 0.5 0.208" rpy="0 0 0"/>
     <axis xyz="0 1 0"/>
-    <dynamics damping="2.5" friction="3000.0"/>  <!-- Increased friction for heavier wing -->
+    <dynamics damping="2.5" friction="10.0"/>  <!-- Lower friction; wing mass/inertia + aero carry the load -->
     <sensor name="left_wing_ft" type="force_torque">
       <update_rate>1</update_rate>
@@ -266,9 +260,9 @@
       <topic>/marid/left_wing/wrench</topic>
     </sensor>
-    <limit lower="-0.5236" upper="0.5236" effort="10" velocity="1.0"/>  <!-- ±30 degrees -->
+    <limit lower="-0.5236" upper="0.5236" effort="500.0" velocity="1.0"/>  <!-- ±30 degrees; servo-like torque limit -->
   </joint>
   <link name="right_wing">
     <inertial>
-      <origin xyz="-1.72531399 -1.11004875 0.18389363"  rpy="0 0 0"/>
+      <origin xyz="${right_wing_inertial}"  rpy="0 0 0"/>
       <mass value="3.662"/>
       <inertia ixx="0.55" ixy="-0.54" ixz="-0.022" iyy="0.662" iyz="-0.021" izz="1.202"/>
@@ -295,5 +289,5 @@
     <origin xyz="-1.225 -0.5 0.208" rpy="0 0 0"/>
     <axis xyz="0 1 0"/>
-    <dynamics damping="2.5" friction="3000.0"/>  <!-- Increased friction for heavier wing -->
+    <dynamics damping="2.5" friction="10.0"/>  <!-- Lower friction; wing mass/inertia + aero carry the load -->
     <sensor name="right_wing_ft" type="force_torque">
       <update_rate>1</update_rate>
@@ -304,14 +298,14 @@
       <topic>/marid/right_wing/wrench</topic>
     </sensor>
-    <limit lower="-0.5236" upper="0.5236" effort="10" velocity="1.0"/>  <!-- ±30 degrees -->
+    <limit lower="-0.5236" upper="0.5236" effort="500.0" velocity="1.0"/>  <!-- ±30 degrees; servo-like torque limit -->
   </joint>
   <link name="tail_left">
     <inertial>
-      <origin xyz="-2.68157748 0.41201641 0.51410285" rpy="0 0 0"/>
+      <origin xyz="${tail_left_inertial}" rpy="0 0 1.57079632679"/>
       <mass value="0.1664684"/>
       <inertia ixx="0.00053436" ixy="0.0" ixz="-0.0003467078" iyy="0.000704515" iyz="0.0" izz="0.0006567504"/>
     </inertial>
     <visual>
-      <origin xyz="0 0 0" rpy="0 0 0"/>
+      <origin xyz="2.559906840 -0.28129418 -0.38425379" rpy="0 0 0"/>
       <geometry>
         <mesh filename="package://marid_description/meshes_2/tail_left.stl"/>
@@ -322,5 +316,5 @@
     </visual>
     <collision>
-      <origin xyz="0 0 0" rpy="0 0 0"/>
+      <origin xyz="2.559906840 -0.28129418 -0.38425379" rpy="0 0 0"/>
       <geometry>
         <mesh filename="package://marid_description/meshes_2/tail_left.stl"/>
@@ -331,7 +325,7 @@
     <parent link="main_tail"/>
     <child link="tail_left"/>
-    <origin xyz="0 0 0" rpy="0 0 0"/>
-    <axis xyz="0.7071 0 -0.7071"/>
-    <dynamics damping="2.5" friction="3000.0"/>  <!-- Lock for aero at high speed; rotation only via actuation -->
+    <origin xyz="-2.559906840 0.28129418 0.38425379" rpy="0 0 0"/>
+    <axis xyz="0 0.7071 0.7071"/>
+    <dynamics damping="2.5" friction="10.0"/>  <!-- Lower friction; tail mass/inertia + aero carry the load -->
     <sensor name="left_tail_ft" type="force_torque">
       <update_rate>1</update_rate>
@@ -342,14 +336,14 @@
       <topic>/marid/left_tail/wrench</topic>
     </sensor>
-    <limit lower="-0.5236" upper="0.5236" effort="10" velocity="1.0"/>  <!-- ±30 degrees -->
+    <limit lower="-0.5236" upper="0.5236" effort="500.0" velocity="1.0"/>  <!-- ±30 degrees; servo-like torque limit -->
   </joint>
   <link name="tail_right">
     <inertial>
-      <origin xyz="-2.68157748 -0.41201641 0.51410285" rpy="0 0 0"/>
+      <origin xyz="${tail_right_inertial}" rpy="0 0 1.57079632679"/>
       <mass value="0.1664684"/>
       <inertia ixx="0.00053436" ixy="0.0" ixz="0.0003467078" iyy="0.000704515" iyz="0.0" izz="0.0006567504"/>
     </inertial>
     <visual>
-      <origin xyz="0 0 0" rpy="0 0 0"/>
+      <origin xyz="2.559906840 0.28129418 -0.38425379" rpy="0 0 0"/>
       <geometry>
         <mesh filename="package://marid_description/meshes_2/tail_right.stl"/>
@@ -360,5 +354,5 @@
     </visual>
     <collision>
-      <origin xyz="0 0 0" rpy="0 0 0"/>
+      <origin xyz="2.559906840 0.28129418 -0.38425379" rpy="0 0 0"/>
       <geometry>
         <mesh filename="package://marid_description/meshes_2/tail_right.stl"/>
@@ -369,7 +363,7 @@
     <parent link="main_tail"/>
     <child link="tail_right"/>
-    <origin xyz="0 0 0" rpy="0 0 0"/>
-    <axis xyz="0.7071 0 0.7071"/>
-    <dynamics damping="2.5" friction="3000.0"/>  <!-- Lock for aero at high speed; rotation only via actuation -->
+    <origin xyz="-2.559906840 -0.28129418 0.38425379" rpy="0 0 0"/>
+    <axis xyz="0 0.7071 -0.7071"/>
+    <dynamics damping="2.5" friction="10.0"/>  <!-- Lower friction; tail mass/inertia + aero carry the load -->
     <sensor name="right_tail_ft" type="force_torque">
       <update_rate>1</update_rate>
@@ -380,5 +374,5 @@
       <topic>/marid/right_tail/wrench</topic>
     </sensor>
-    <limit lower="-0.5236" upper="0.5236" effort="10" velocity="1.0"/>  <!-- ±30 degrees -->
+    <limit lower="-0.5236" upper="0.5236" effort="500.0" velocity="1.0"/>  <!-- ±30 degrees; servo-like torque limit -->
   </joint>
   <link name="imu_link">
@@ -479,5 +473,5 @@
   <link name="thruster_L">
     <inertial>
-      <origin xyz="-1.20 -0.3 0.50" rpy="0 0 0"/>
+      <origin xyz="0 0 0" rpy="0 0 0"/>
       <mass value="0.05"/>
       <inertia ixx="1e-5" ixy="0" ixz="0" iyy="1e-5" iyz="0" izz="1e-5"/>
@@ -494,5 +488,5 @@
   <link name="thruster_R">
     <inertial>
-      <origin xyz="-1.20 0.3 0.50" rpy="0 0 0"/>
+      <origin xyz="0 0 0" rpy="0 0 0"/>
       <mass value="0.05"/>
       <inertia ixx="1e-5" ixy="0" ixz="0" iyy="1e-5" iyz="0" izz="1e-5"/>

File: src/marid_description/urdf/marid_new_gazebo.xacro (robot description, xacro)
@@ -52,12 +52,12 @@
         <maxVel>0.2</maxVel>
     </gazebo>
-        <gazebo reference="rear_wheel">
-          <mu1>0.9</mu1>
-          <mu2>0.9</mu2>
-          <kp>2e5</kp>
-          <kd>2e3</kd>
-          <minDepth>0.001</minDepth>
-          <maxVel>0.2</maxVel>
-      </gazebo>
+    <gazebo reference="rear_wheel">
+        <mu1>0.9</mu1>
+        <mu2>0.9</mu2>
+        <kp>2e5</kp>
+        <kd>2e3</kd>
+        <minDepth>0.001</minDepth>
+        <maxVel>0.2</maxVel>
+    </gazebo>
     <!-- Aircraft-level aerodynamic model: AdvancedLiftDrag (single plugin) -->
     <gazebo>
@@ -100,5 +100,5 @@
             <Cema_stall>0</Cema_stall>
             <!-- Aerodynamic reference geometry (scaled for larger MARID airframe) -->
-            <cp>0 0 0</cp>          <!-- Aerodynamic center in base_link_front frame -->
+            <cp>-1.876 0 0.306</cp>          <!-- Aerodynamic center in base_link_front frame -->
             <area>2.0</area>        <!-- Reference area (m²) - scaled up for bigger drone -->
             <mac>0.35</mac>         <!-- Mean aerodynamic chord (m) - scaled for bigger drone -->
@@ -115,5 +115,5 @@
                 <name>left_wing_joint</name>
                 <index>0</index>
-                <direction>1</direction>   <!-- Match right wing: both wings -1 to fix right-side lift bias -->
+                <direction>1</direction>   <!-- Same direction as right wing; differential deflection gives roll -->
                 <!-- Coefficients copied from reference servo_0 as a starting point -->
                 <CL_ctrl>2.2</CL_ctrl>
@@ -136,5 +136,5 @@
                 <Cen_ctrl>-0.01</Cen_ctrl>
             </control_surface>
-            <!-- Left tail surface (V-tail); direction matches reference servo_2 -->
+            <!-- Left tail surface (V-tail); tuned for MARID V-tail geometry -->
             <control_surface>
                 <name>tail_left_joint</name>
@@ -143,18 +143,18 @@
                 <CL_ctrl>0.4</CL_ctrl>
                 <CD_ctrl>0.02</CD_ctrl>
-                <Cem_ctrl>-0.25</Cem_ctrl>
+                <Cem_ctrl>0.25</Cem_ctrl>
                 <Cen_ctrl>0.10</Cen_ctrl>
                 <CY_ctrl>0.00</CY_ctrl>
                 <Cell_ctrl>0.00</Cell_ctrl>
             </control_surface>
-            <!-- Right tail surface (V-tail); direction matches reference servo_3 -->
+            <!-- Right tail surface (V-tail); tuned so symmetric deflection gives mostly pitch, differential gives yaw -->
             <control_surface>
                 <name>tail_right_joint</name>
                 <index>3</index>
-                <direction>-1</direction>
+                <direction>1</direction>
                 <CL_ctrl>0.4</CL_ctrl>
                 <CD_ctrl>0.02</CD_ctrl>
-                <Cem_ctrl>-0.25</Cem_ctrl>
-                <Cen_ctrl>-0.10</Cen_ctrl>
+                <Cem_ctrl>0.25</Cem_ctrl>   <!-- With direction=1, Cem matches left tail so symmetric deflection adds pitch -->
+                <Cen_ctrl>-0.10</Cen_ctrl>  <!-- With direction=1, Cen opposes left tail so symmetric deflection cancels yaw -->
                 <CY_ctrl>0.00</CY_ctrl>
                 <Cell_ctrl>0.00</Cell_ctrl>
@@ -192,5 +192,5 @@
         </plugin>
     </gazebo>
-    <!-- ===== CENTER: Thruster plugin (force in N) - scaled for bigger drone, CCW rotation ===== -->
+    <!-- ===== CENTER: Thruster plugin (force in N) - scaled for bigger drone; rotation per thrust_coefficient sign (see comment) ===== -->
     <gazebo>
         <plugin filename="libgz-sim8-thruster-system.so" name="gz::sim::systems::Thruster">
@@ -243,5 +243,5 @@
     </gazebo>
     <!-- ===== JOINT POSITION CONTROLLERS FOR CONTROL SURFACES ===== -->
-    <!-- P-gain raised to overcome 150 N·m joint friction (wings/tails) for bigger drone -->
+    <!-- P-gain chosen so controllers can hold wings/tails stiff against aero and gravity with ~10 N·m joint friction -->
     <!-- Left Wing Position Controller -->
     <gazebo>
@@ -249,5 +249,5 @@
                 name="gz::sim::systems::JointPositionController">
             <joint_name>left_wing_joint</joint_name>
-            <p_gain>80.0</p_gain>
+            <p_gain>600.0</p_gain>
             <topic>/model/marid/joint/left_wing_joint/cmd_pos</topic>
         </plugin>
@@ -258,5 +258,5 @@
                 name="gz::sim::systems::JointPositionController">
             <joint_name>right_wing_joint</joint_name>
-            <p_gain>80.0</p_gain>
+            <p_gain>600.0</p_gain>
             <topic>/model/marid/joint/right_wing_joint/cmd_pos</topic>
         </plugin>
@@ -267,5 +267,5 @@
                 name="gz::sim::systems::JointPositionController">
             <joint_name>tail_left_joint</joint_name>
-            <p_gain>80.0</p_gain>
+            <p_gain>280.0</p_gain>
             <topic>/model/marid/joint/tail_left_joint/cmd_pos</topic>
         </plugin>
@@ -276,5 +276,5 @@
                 name="gz::sim::systems::JointPositionController">
             <joint_name>tail_right_joint</joint_name>
-            <p_gain>80.0</p_gain>
+            <p_gain>280.0</p_gain>
             <topic>/model/marid/joint/tail_right_joint/cmd_pos</topic>
         </plugin>
