Commit message: Tune MARID aero controls and lift-off parameters
- Adjust front wing AdvancedLiftDrag control-surface signs.
- Review V-tail Cen_ctrl and overall sign patterns to ensure symmetric pitch and differential yaw are accurate.
-  Replace detailed wheel meshes with cylinder primitives to avoid non‑smooth triangulated CAD geometry and improve contact stability in Gazebo.
- Retune thrust logic: increase maximum available thrust in the Gazebo thruster plugin and guidance tracker, and adjust desired cruise speed / target velocity so physics‑based thrust can command higher forces.

File: src/marid_description/urdf/marid_new.urdf.xacro (robot description, xacro)
@@ -105,14 +105,16 @@
     </visual>
     <collision>
-      <origin xyz="0.525 -0.20786886 0.09000082" rpy="0 0 0"/>
-      <geometry>
-        <mesh filename="package://marid_description/meshes_2/front_left_tire.stl"/>
-      </geometry>
-    </collision>
-  </link>
-  <joint name="left_front_wheel_joint" type="fixed">
+      <origin xyz="0 0 0" rpy="1.5708 0 0"/>
+      <geometry>
+        <cylinder radius="0.089" length="0.05"/>
+      </geometry>
+    </collision>
+  </link>
+  <joint name="left_front_wheel_joint" type="continuous">
     <parent link="left_front_wheel_arm"/>
     <child link="left_front_wheel"/>
     <origin xyz="-0.525 0.20786886 -0.09000082" rpy="0 0 0"/>
+    <axis xyz="0 1 0"/>  <!-- Wheel rotation around own axle (parallel to world Y) -->
+    <dynamics damping="0.01" friction="0.0"/>
   </joint>
   <link name="right_front_wheel">
@@ -132,14 +134,16 @@
     </visual>
     <collision>
-      <origin xyz="0.525 0.20786886 0.09000082" rpy="0 0 0"/>
-      <geometry>
-        <mesh filename="package://marid_description/meshes_2/front_right_tire.stl"/>
-      </geometry>
-    </collision>
-  </link>
-  <joint name="right_front_wheel_joint" type="fixed">
+      <origin xyz="0 0 0" rpy="1.5708 0 0"/>
+      <geometry>
+        <cylinder radius="0.089" length="0.05"/>
+      </geometry>
+    </collision>
+  </link>
+  <joint name="right_front_wheel_joint" type="continuous">
     <parent link="right_front_wheel_arm"/>
     <child link="right_front_wheel"/>
     <origin xyz="-0.525 -0.20786886 -0.09000082" rpy="0 0 0"/>
+    <axis xyz="0 1 0"/>  <!-- Wheel rotation around own axle (parallel to world Y) -->
+    <dynamics damping="0.01" friction="0.0"/>
   </joint>
   <link name="rear_wheel_arm">
@@ -186,14 +190,16 @@
     </visual>
     <collision>
-      <origin xyz="2.475 0 0.02500082" rpy="0 0 0"/>
-      <geometry>
-        <mesh filename="package://marid_description/meshes_2/rear_tire.stl"/>
-      </geometry>
-    </collision>
-  </link>
-  <joint name="rear_wheel_joint" type="fixed">
+      <origin xyz="0 0 0" rpy="1.5708 0 0"/>
+      <geometry>
+        <cylinder radius="0.08" length="0.05"/>
+      </geometry>
+    </collision>
+  </link>
+  <joint name="rear_wheel_joint" type="continuous">
     <parent link="rear_wheel_arm"/>
     <child link="rear_wheel"/>
     <origin xyz="-2.475 0 -0.02500082" rpy="0 0 0"/>
+    <axis xyz="0 1 0"/>  <!-- Wheel rotation around own axle (parallel to world Y) -->
+    <dynamics damping="0.01" friction="0.0"/>
   </joint>
   <link name="main_tail">

File: src/marid_description/urdf/marid_new_gazebo.xacro (robot description, xacro)
@@ -115,12 +115,12 @@
                 <name>left_wing_joint</name>
                 <index>0</index>
-                <direction>1</direction>   <!-- Same direction as right wing; differential deflection gives roll -->
+                <direction>-1</direction>   <!-- Same direction as right wing; differential deflection gives roll -->
                 <!-- Coefficients copied from reference servo_0 as a starting point -->
                 <CL_ctrl>2.2</CL_ctrl>
-                <CD_ctrl>0.06</CD_ctrl>
-                <Cem_ctrl>-0.35</Cem_ctrl>
-                <Cell_ctrl>-0.05</Cell_ctrl>
+                <CD_ctrl>0.08</CD_ctrl>
+                <Cem_ctrl>0.45</Cem_ctrl>
+                <Cell_ctrl>0.05</Cell_ctrl>
                 <CY_ctrl>0.00</CY_ctrl>
-                <Cen_ctrl>0.01</Cen_ctrl>
+                <Cen_ctrl>-0.01</Cen_ctrl>
             </control_surface>
             <!-- Right wing; direction matches reference servo_1 -->
@@ -128,11 +128,11 @@
                 <name>right_wing_joint</name>
                 <index>1</index>
-                <direction>1</direction>
+                <direction>-1</direction>
                 <CL_ctrl>2.2</CL_ctrl>
-                <CD_ctrl>0.06</CD_ctrl>
-                <Cem_ctrl>-0.35</Cem_ctrl>
-                <Cell_ctrl>0.05</Cell_ctrl>
+                <CD_ctrl>0.08</CD_ctrl>
+                <Cem_ctrl>0.45</Cem_ctrl>
+                <Cell_ctrl>-0.05</Cell_ctrl>
                 <CY_ctrl>0.00</CY_ctrl>
-                <Cen_ctrl>-0.01</Cen_ctrl>
+                <Cen_ctrl>0.01</Cen_ctrl>
             </control_surface>
             <!-- Left tail surface (V-tail); tuned for MARID V-tail geometry -->
@@ -144,5 +144,5 @@
                 <CD_ctrl>0.02</CD_ctrl>
                 <Cem_ctrl>0.25</Cem_ctrl>
-                <Cen_ctrl>0.10</Cen_ctrl>
+                <Cen_ctrl>-0.05</Cen_ctrl>
                 <CY_ctrl>0.00</CY_ctrl>
                 <Cell_ctrl>0.00</Cell_ctrl>
@@ -156,5 +156,5 @@
                 <CD_ctrl>0.02</CD_ctrl>
                 <Cem_ctrl>0.25</Cem_ctrl>   <!-- With direction=1, Cem matches left tail so symmetric deflection adds pitch -->
-                <Cen_ctrl>-0.10</Cen_ctrl>  <!-- With direction=1, Cen opposes left tail so symmetric deflection cancels yaw -->
+                <Cen_ctrl>0.05</Cen_ctrl>  <!-- With direction=1, Cen opposes left tail so symmetric deflection cancels yaw -->
                 <CY_ctrl>0.00</CY_ctrl>
                 <Cell_ctrl>0.00</Cell_ctrl>

Commit message: Improve gazebo sensor pipelines and imu odometry debugging outputs
- Fix LiDAR Gazebo-to-ROS bridge mapping to the correct point cloud source, restoring /lidar/scan PointCloud2 visibility in ROS/RViz.
- Enhance marid_odom_pub with barometer-assisted altitude fusion for improved vertical stability.
- Publish IMU-odometry TF on a separate child frame to compare IMU-derived motion against EKF/ground-truth without transform conflicts.
- Restore camera output path end-to-end (Gazebo sensor → bridge → ROS image topic) and expose camera feed in Gazebo GUI.
- Update empty.sdf GUI/world configuration to support 3D scene + camera + inspection panels for faster debugging workflows.

File: src/marid_description/urdf/marid_new.urdf.xacro (robot description, xacro)
@@ -266,5 +266,5 @@
       <topic>/marid/left_wing/wrench</topic>
     </sensor>
-    <limit lower="-0.5236" upper="0.5236" effort="500.0" velocity="1.0"/>  <!-- ±30 degrees; servo-like torque limit -->
+    <limit lower="-0.075" upper="0.075" effort="700.0" velocity="1.0"/>  <!-- ±30 degrees; servo-like torque limit -->
   </joint>
   <link name="right_wing">
@@ -304,5 +304,5 @@
       <topic>/marid/right_wing/wrench</topic>
     </sensor>
-    <limit lower="-0.5236" upper="0.5236" effort="500.0" velocity="1.0"/>  <!-- ±30 degrees; servo-like torque limit -->
+    <limit lower="-0.075" upper="0.075" effort="700.0" velocity="1.0"/>  <!-- ±30 degrees; servo-like torque limit -->
   </joint>
   <link name="tail_left">
@@ -342,5 +342,5 @@
       <topic>/marid/left_tail/wrench</topic>
     </sensor>
-    <limit lower="-0.5236" upper="0.5236" effort="500.0" velocity="1.0"/>  <!-- ±30 degrees; servo-like torque limit -->
+    <limit lower="-0.1" upper="0.1" effort="500.0" velocity="1.0"/>  <!-- ±30 degrees; servo-like torque limit -->
   </joint>
   <link name="tail_right">
@@ -380,5 +380,5 @@
       <topic>/marid/right_tail/wrench</topic>
     </sensor>
-    <limit lower="-0.5236" upper="0.5236" effort="500.0" velocity="1.0"/>  <!-- ±30 degrees; servo-like torque limit -->
+    <limit lower="-0.1" upper="0.1" effort="500.0" velocity="1.0"/>  <!-- ±30 degrees; servo-like torque limit -->
   </joint>
   <link name="imu_link">
@@ -574,5 +574,6 @@
     <child link="camera_link"/>
     <!-- Nose mount, forward-looking -->
-    <origin xyz="0 0 0" rpy="0 0 0"/>
+    <!-- Rotate camera 15 degrees around Y axis (pitch up, CCW in URDF rpy) -->
+    <origin xyz="0 0 0" rpy="0 0.261799 0"/>
   </joint>
     <!-- Nose propeller (MulticopterMotorModel: command motor speed rad/s on command/motor_speed_nose) -->

File: src/marid_description/urdf/marid_new_gazebo.xacro (robot description, xacro)
@@ -117,5 +117,5 @@
                 <direction>-1</direction>   <!-- Same direction as right wing; differential deflection gives roll -->
                 <!-- Coefficients copied from reference servo_0 as a starting point -->
-                <CL_ctrl>2.2</CL_ctrl>
+                <CL_ctrl>2.0</CL_ctrl>
                 <CD_ctrl>0.08</CD_ctrl>
                 <Cem_ctrl>0.45</Cem_ctrl>
@@ -129,5 +129,5 @@
                 <index>1</index>
                 <direction>-1</direction>
-                <CL_ctrl>2.2</CL_ctrl>
+                <CL_ctrl>2.0</CL_ctrl>
                 <CD_ctrl>0.08</CD_ctrl>
                 <Cem_ctrl>0.45</Cem_ctrl>
@@ -141,5 +141,5 @@
                 <index>2</index>
                 <direction>1</direction>
-                <CL_ctrl>0.4</CL_ctrl>
+                <CL_ctrl>0.2</CL_ctrl>
                 <CD_ctrl>0.02</CD_ctrl>
                 <Cem_ctrl>0.25</Cem_ctrl>
@@ -153,5 +153,5 @@
                 <index>3</index>
                 <direction>1</direction>
-                <CL_ctrl>0.4</CL_ctrl>
+                <CL_ctrl>0.2</CL_ctrl>
                 <CD_ctrl>0.02</CD_ctrl>
                 <Cem_ctrl>0.25</Cem_ctrl>   <!-- With direction=1, Cem matches left tail so symmetric deflection adds pitch -->
@@ -483,5 +483,5 @@
         <odom_frame>odom</odom_frame>
         <robot_base_frame>base_link_front</robot_base_frame>
-        <publish_tf>false</publish_tf>
+        <publish_tf>true</publish_tf>
       </plugin>
     </gazebo>

Commit message: Improve GPS-denied localization with airspeed dead reckoning
Core localization improvements (marid_odom_pub.py):
- Replace IMU double-integration velocity with airspeed complementary filter:
  airspeed rotated by IMU attitude gives velocity via single integration,
  dramatically reducing position drift vs double-integrating acceleration
- Replace FAST-LIO hard position reset with configurable soft correction
  (fastlio_position_weight=0.3) so airspeed dead reckoning owns position
  between LiDAR updates rather than blindly following FAST-LIO drift
- Disable wind correction by default in sim: wind estimator was circular
  (used EKF/Gazebo ground truth), effectively injecting GPS data into the
  GPS-denied estimator and acting as artificial headwind/tailwind

Sensor pipeline fixes:
- Add /airspeed bridge to ros_gz_bridge (was missing entirely, forcing
  airspeed_converter to poll via subprocess with up to 1s latency)
- Rewrite airspeed_converter.py as a proper ROS2 subscriber to
  ros_gz_interfaces/msg/AirSpeed — event-driven at sensor rate, zero
  subprocess overhead
- Fix wind_estimator.py frame bug: EKF twist.twist.linear is in body
  frame, not odom frame; rotation to odom frame was missing before
  computing v_wind = v_ground - v_air
- Reduce FAST-LIO IMU covariance acc_cov/gyr_cov 0.1→0.01 to weight
  IMU more heavily during flat-ground scan-matching degeneracy

Sensor/HUD improvements (pre-existing staged changes):
- Widen camera HUD horizon line and add roll-aligned pitch bars
- Register lidar_time_field.py in CMakeLists and launch it from
  fast_lio.launch.py to inject per-point timestamps Gazebo omits
- Increase thrust_gain default 250→500 in cmd_vel_to_wings

File: src/marid_description/urdf/marid_new.urdf.xacro (robot description, xacro)
@@ -266,5 +266,5 @@
       <topic>/marid/left_wing/wrench</topic>
     </sensor>
-    <limit lower="-0.075" upper="0.075" effort="700.0" velocity="1.0"/>  <!-- ±30 degrees; servo-like torque limit -->
+    <limit lower="-0.15" upper="0.15" effort="700.0" velocity="1.0"/>  <!-- ±30 degrees; servo-like torque limit -->
   </joint>
   <link name="right_wing">
@@ -304,5 +304,5 @@
       <topic>/marid/right_wing/wrench</topic>
     </sensor>
-    <limit lower="-0.075" upper="0.075" effort="700.0" velocity="1.0"/>  <!-- ±30 degrees; servo-like torque limit -->
+    <limit lower="-0.15" upper="0.15" effort="700.0" velocity="1.0"/>  <!-- ±30 degrees; servo-like torque limit -->
   </joint>
   <link name="tail_left">
@@ -342,5 +342,5 @@
       <topic>/marid/left_tail/wrench</topic>
     </sensor>
-    <limit lower="-0.1" upper="0.1" effort="500.0" velocity="1.0"/>  <!-- ±30 degrees; servo-like torque limit -->
+    <limit lower="-0.25" upper="0.25" effort="500.0" velocity="1.0"/>  <!-- ±30 degrees; servo-like torque limit -->
   </joint>
   <link name="tail_right">
@@ -380,5 +380,5 @@
       <topic>/marid/right_tail/wrench</topic>
     </sensor>
-    <limit lower="-0.1" upper="0.1" effort="500.0" velocity="1.0"/>  <!-- ±30 degrees; servo-like torque limit -->
+    <limit lower="-0.25" upper="0.25" effort="500.0" velocity="1.0"/>  <!-- ±30 degrees; servo-like torque limit -->
   </joint>
   <link name="imu_link">
@@ -451,5 +451,5 @@
     <parent link="base_link_front"/>
     <child link="lidar_link"/>
-    <origin xyz="0 0.2 0.05" rpy="0 0 0"/>  <!-- LIDAR offset from base (Y right, Z up) -->
+    <origin xyz="0 0 0.05" rpy="0 0 0"/>  <!-- LIDAR offset from base (Y right, Z up) -->
   </joint>
   <link name="pitot_link">
@@ -555,5 +555,5 @@
     </inertial>
     <visual>
-      <origin xyz="-1 0 1" rpy="0 0 0"/>
+      <origin xyz="-0.025 0 .25" rpy="0 0 0"/>
       <geometry>
         <box size="0.02 0.06 0.02"/>
@@ -575,5 +575,5 @@
     <!-- Nose mount, forward-looking -->
     <!-- Rotate camera 15 degrees around Y axis (pitch up, CCW in URDF rpy) -->
-    <origin xyz="0 0 0" rpy="0 0.261799 0"/>
+    <origin xyz="0 0 0" rpy="0 0 0"/>
   </joint>
     <!-- Nose propeller (MulticopterMotorModel: command motor speed rad/s on command/motor_speed_nose) -->

Commit message: Add wheel odometry fusion and forward camera lateral velocity estimator
  Fuse /wheel/odometry into marid_odom_pub for ground taxiing: wheel odom
  owns XY position when sonar AGL <= 0.30m, gating FAST-LIO position writes
  and optical flow dead-reckoning while on the ground.

  Fix Gazebo joint states topic mismatch: robot_state_publisher and
  wheel_odometry_node were subscribing to /joint_states but the gz-ros2
  bridge publishes to /world/empty/model/marid/joint_state. Added remappings
  so wheel TF frames animate correctly and wheel velocities are received.

  Add forward_flow_estimator.py: Lucas-Kanade sparse tracking with IMU gyro
  compensation extracts lateral (vy) and vertical (vz) body-frame velocity
  from the forward camera. Depth is estimated as depth_scale * altitude.
  Fused into marid_odom_pub above 1m AGL to constrain lateral drift during
  flight where the downward optical flow camera is inactive.

File: src/marid_description/urdf/marid_new.urdf.xacro (robot description, xacro)
@@ -577,4 +577,40 @@
     <origin xyz="0 0 0" rpy="0 0 0"/>
   </joint>
+  <!-- Optical Flow Camera - belly mount, downward facing -->
+  <link name="optical_flow_link">
+    <inertial>
+      <mass value="0.01"/>
+      <origin xyz="0 0 0"/>
+      <inertia ixx="1e-6" iyy="1e-6" izz="1e-6" ixy="0" ixz="0" iyz="0"/>
+    </inertial>
+    <visual>
+      <origin xyz="0 0 0" rpy="0 0 0"/>
+      <geometry><box size="0.02 0.02 0.01"/></geometry>
+      <material name="of_gray"><color rgba="0.5 0.5 0.5 1.0"/></material>
+    </visual>
+    <collision>
+      <origin xyz="0 0 0" rpy="0 0 0"/>
+      <geometry><box size="0.02 0.02 0.01"/></geometry>
+    </collision>
+  </link>
+  <!-- rpy="0 1.5708 0": pitch +90° rotates sensor +X to body -Z (downward) -->
+  <joint name="optical_flow_joint" type="fixed">
+    <parent link="base_link_front"/>
+    <child link="optical_flow_link"/>
+    <origin xyz="-0.5 0 0.1" rpy="0 1.5708 0"/>
+  </joint>
+  <!-- Sonar Rangefinder - belly mount, downward facing -->
+  <link name="sonar_link">
+    <inertial>
+      <mass value="0.005"/>
+      <origin xyz="0 0 0"/>
+      <inertia ixx="1e-7" iyy="1e-7" izz="1e-7" ixy="0" ixz="0" iyz="0"/>
+    </inertial>
+  </link>
+  <joint name="sonar_joint" type="fixed">
+    <parent link="base_link_front"/>
+    <child link="sonar_link"/>
+    <origin xyz="-0.5 0 0.1" rpy="0 1.5708 0"/>
+  </joint>
     <!-- Nose propeller (MulticopterMotorModel: command motor speed rad/s on command/motor_speed_nose) -->
   <link name="nose_prop">

File: src/marid_description/urdf/marid_new_gazebo.xacro (robot description, xacro)
@@ -1,4 +1,12 @@
 <?xml version="1.0"?>
 <robot name="marid" xmlns:xacro="http://www.ros.org/wiki/xacro">
+    <!-- Joint state publisher — exposes all joint positions and velocities on
+         /world/empty/model/marid/joint_state (gz.msgs.Model), bridged to
+         /joint_states (sensor_msgs/JointState) for the wheel odometry node. -->
+    <gazebo>
+      <plugin filename="gz-sim-joint-state-publisher-system"
+              name="gz::sim::systems::JointStatePublisher">
+      </plugin>
+    </gazebo>
     <!-- WIND ENABLE -->
     <gazebo>
@@ -467,4 +475,67 @@
       </sensor>
     </gazebo>
+    <!-- Optical Flow Camera - downward facing, 320x240, 30 Hz -->
+    <!-- Joint rpy="0 1.5708 0" makes sensor +X point down, so camera looks at ground -->
+    <gazebo reference="optical_flow_link">
+      <sensor name="optical_flow_camera" type="camera">
+        <always_on>true</always_on>
+        <update_rate>30</update_rate>
+        <topic>/optical_flow/camera</topic>
+        <gz_frame_id>optical_flow_link</gz_frame_id>
+        <camera>
+          <horizontal_fov>1.047</horizontal_fov>  <!-- 60 deg -->
+          <image>
+            <width>320</width>
+            <height>240</height>
+            <format>R8G8B8</format>
+          </image>
+          <clip>
+            <near>0.05</near>
+            <far>15</far>
+          </clip>
+          <noise>
+            <type>gaussian</type>
+            <mean>0.0</mean>
+            <stddev>1.5</stddev>
+          </noise>
+        </camera>
+      </sensor>
+    </gazebo>
+    <!-- Sonar Rangefinder - single downward beam, 0.05-5 m, 25 Hz -->
+    <!-- Joint rpy="0 1.5708 0" makes sensor +X point down; lidar emits along +X -->
+    <gazebo reference="sonar_link">
+      <sensor name="sonar" type="gpu_lidar">
+        <always_on>true</always_on>
+        <update_rate>25</update_rate>
+        <topic>/sonar/scan</topic>
+        <gz_frame_id>sonar_link</gz_frame_id>
+        <ray>
+          <scan>
+            <horizontal>
+              <samples>1</samples>
+              <resolution>1</resolution>
+              <min_angle>0</min_angle>
+              <max_angle>0</max_angle>
+            </horizontal>
+            <vertical>
+              <samples>1</samples>
+              <resolution>1</resolution>
+              <min_angle>0</min_angle>
+              <max_angle>0</max_angle>
+            </vertical>
+          </scan>
+          <range>
+            <min>0.05</min>
+            <max>5.0</max>
+            <resolution>0.01</resolution>
+          </range>
+          <noise>
+            <type>gaussian</type>
+            <mean>0.0</mean>
+            <stddev>0.02</stddev>
+          </noise>
+        </ray>
+      </sensor>
+    </gazebo>
     <!-- Pose Publisher Plugin - publishes model pose for localization -->
     <gazebo reference="base_link_front">
