Commit message: Add ESKF, sun sensor, joystick teleop, and fix aerodynamic pitch instability
  Description:
  GPS-denied estimation — ESKF (marid_odom_pub.py):
  - Implement full Error-State Kalman Filter (MARIDESKF class) with two
    propagation modes: "imu" (δx ∈ ℝ¹²) and "physics" (δx ∈ ℝ¹⁴)
  - Physics mode augments state with drag coefficient (kd) and H2 fuel
    mass (mh2), using aerodynamic model mirroring AdvancedLiftDrag plugin
    (CL0, CLa, wing area, control surface CL_ctrl, stall model)
  - IMU mode: standard specific-force prediction + gyro integration
  - Chi-squared outlier gating, quaternion [x,y,z,w] ENU convention

  Sun sensor simulator (sun_sensor_sim.py — new):
  - Computes solar azimuth/elevation from sim time + lat/lon (MARID datum)
  - Rotates sun ENU vector into body frame via ground-truth Gazebo pose
  - Publishes /sun_sensor/sun_vector_body and azimuth/elevation for
    heading correction independent of estimation pipeline

  State error monitor (vx_error_monitor.py):
  - Expanded from vx-only to full 6-DOF: position (x,y,z) + velocity
    (vx,vy,vz), with per-channel ground-truth vs estimate comparison
  - Separate min_pos / min_speed percentage denominators

  Localization launch (local_localization.launch.py):
  - Wire in ESKF node (use_eskf: true, eskf_mode: physics) and
    sun_sensor_sim node

  Guidance improvements:
  - marid_ai_guidance: altitude gate with configurable tolerance +
    stable-hold duration before transitioning climb → navigate phase
  - marid_guidance_tracker: fix thrust formula — base_thrust = drag
    (fixed-wing equilibrium), not drag + weight (helicopter logic);
    disable yaw differential (yaw handled by attitude controller tail)

  Joystick incremental teleop (joy_incrementer.py — new):
  - Press-based control: Y/A ±10N thrust, button 6 halve thrust + zero
    wings, button 7 preset 2165N, D-pad ±0.02 rad v-tail, X/B ±0.02 rad
    front wing AOA; edge detection prevents repeat-fire on hold
  - Thrust published at 20 Hz directly to Gazebo thruster joint,
    decoupled from cmd_vel pipeline
  - cmd_vel_to_wings: remove thrust, blend vtail/wing offsets additively

  Aerodynamic stability (marid_new_gazebo.xacro):
  - Flip Cema: +0.463966 → -0.463966 (pitch-unstable → stable; CP was
    6.5 cm ahead of CG, -18.6% static margin)
  - Move aerodynamic center aft: -1.876 m → -1.98 m (+11% MAC margin)
  - Reduce barometer noise: 5.0 Pa → 0.5 Pa stddev (5 Pa ≈ 0.4 m
    altitude error at 1σ; was triggering false airborne on runway)

  Attitude controller (marid_attitude_controller.py):
  - Gate airborne detection on altitude AND speed (>20 m/s) to prevent
    pitch activation from baro noise during ground roll

  URDF / world:
  - Expand wing joint limits: ±0.25 → ±0.35 rad for greater AOA range
  - Update wind direction vector in empty.sdf

File: src/marid_description/urdf/marid_new.urdf.xacro (robot description, xacro)
@@ -342,5 +342,5 @@
       <topic>/marid/left_tail/wrench</topic>
     </sensor>
-    <limit lower="-0.25" upper="0.25" effort="500.0" velocity="1.0"/>  <!-- ±30 degrees; servo-like torque limit -->
+    <limit lower="-0.35" upper="0.35" effort="500.0" velocity="1.0"/>  <!-- ±20 degrees; servo-like torque limit -->
   </joint>
   <link name="tail_right">
@@ -380,5 +380,5 @@
       <topic>/marid/right_tail/wrench</topic>
     </sensor>
-    <limit lower="-0.25" upper="0.25" effort="500.0" velocity="1.0"/>  <!-- ±30 degrees; servo-like torque limit -->
+    <limit lower="-0.35" upper="0.35" effort="500.0" velocity="1.0"/>  <!-- ±20 degrees; servo-like torque limit -->
   </joint>
   <link name="imu_link">

File: src/marid_description/urdf/marid_new_gazebo.xacro (robot description, xacro)
@@ -81,5 +81,5 @@
             <CD0>0.04</CD0>
             <Cem0>-0.03</Cem0>   <!-- Flipped for X-forward: reduce nose-down tendency -->
-            <Cema>0.463966</Cema>
+            <Cema>-0.463966</Cema>
             <CYb>-0.258244</CYb>
             <Cellb>-0.03925</Cellb>
@@ -108,5 +108,5 @@
             <Cema_stall>0</Cema_stall>
             <!-- Aerodynamic reference geometry (scaled for larger MARID airframe) -->
-            <cp>-1.876 0 0.306</cp>          <!-- Aerodynamic center in base_link_front frame -->
+            <cp>-1.98 0 0.306</cp>            <!-- Aerodynamic center: moved aft of CG (~-1.941m) for +11% MAC static margin -->
             <area>2.0</area>        <!-- Reference area (m²) - scaled up for bigger drone -->
             <mac>0.35</mac>         <!-- Mean aerodynamic chord (m) - scaled for bigger drone -->
@@ -123,5 +123,5 @@
                 <name>left_wing_joint</name>
                 <index>0</index>
-                <direction>-1</direction>   <!-- Same direction as right wing; differential deflection gives roll -->
+                <direction>-1</direction>   <!-- -1: negative deflection = trailing edge up = increase CL and pitch-up moment -->
                 <!-- Coefficients copied from reference servo_0 as a starting point -->
                 <CL_ctrl>2.0</CL_ctrl>
@@ -431,5 +431,5 @@
             <noise type="gaussian">
               <mean>0.0</mean>
-              <stddev>0.01</stddev>
+              <stddev>5e-8</stddev>
             </noise>
           </x>
@@ -437,5 +437,5 @@
             <noise type="gaussian">
               <mean>0.0</mean>
-              <stddev>0.01</stddev>
+              <stddev>5e-8</stddev>
             </noise>
           </y>
@@ -443,5 +443,5 @@
             <noise type="gaussian">
               <mean>0.0</mean>
-              <stddev>0.01</stddev>
+              <stddev>5e-8</stddev>
             </noise>
           </z>
@@ -471,5 +471,5 @@
         <noise type="gaussian">
           <mean>0.0</mean>
-          <stddev>5.0</stddev>
+          <stddev>0.5</stddev>
         </noise>
       </sensor>
