Commit message: Overhaul ESKF sensor fusion, add ML training pipeline, and expand simulation
  ESKF (marid_odom_pub.py):
  - Add gyro bias bg to state vector (n=15 IMU / n=17 physics); freeze_bg
    in all kinematic updates to prevent velocity/position measurements from
    corrupting bg through cross-covariance
  - Add is_airborne_ 5-tick debounce; fix liftoff vy snap by preserving
    ESKF yaw in ground clamp and gating 2D airspeed constraint on is_airborne_
  - Add update_airspeed_world_velocity: 2D world-frame Va + zero-sideslip
    constraint replacing 1D body-velocity update during airborne flight
  - Add coordinated-turn gyro bias estimator (bg_q, bg_r only; H[yaw]=0)
  - Add sun sensor yaw update; Madgwick bank gate (25x inflation at |roll|>12°)
  - Add P inflation on yaw jump >15° for fast velocity re-convergence
  - Add quaternion divergence gate (fallback to Madgwick when |dot|<0.94)
  - Reduce Madgwick gain 0.3->0.05 to reduce centripetal corruption in turns

  Hardware/simulation:
  - Add 5-hole probe lateral and vertical sensor links to URDF
  - Add terrain world with DEM heightmap pipeline (dem_to_heightmap.py)
  - Option A launch: randomised GPS destination with radius/seed params
  - Joystick teleop: new yaml config, launch file, and joy_incrementer
  - Sun sensor sim: suppress publish when sun below sensor hemisphere
  - Camera HUD: add ESKF vs GT attitude and velocity overlay

  ML pipeline (all new):
  - eskf_gt_logger.py: flight data logger for supervised training
  - eskf_attitude_ff_train.py / eskf_attitude_lstm_train.py: yaw correction models
  - eskf_velocity_lstm_train.py / eskf_position_lstm_train.py: velocity/position models
  - compare_results.py, model_observation.ipynb: analysis tools

  Housekeeping:
  - .gitignore: exclude data/ and data_extended/ binaries
  - Remove stale data/*.npz legacy flight chunks

File: src/marid_description/urdf/marid_new.urdf.xacro (robot description, xacro)
@@ -465,4 +465,30 @@
     <origin xyz="0 0 0" rpy="0 0 0"/>  <!-- Pitot at base origin (tune position for nose airflow) -->
   </joint>
+  <!-- 5-hole probe lateral (body-y): sensor x-axis rotated to align with body +y -->
+  <link name="airspeed_y_link">
+    <inertial>
+      <mass value="0.001"/>
+      <origin xyz="-1.1 0 0.15"/>
+      <inertia ixx="1e-7" iyy="1e-7" izz="1e-7" ixy="0" ixz="0" iyz="0"/>
+    </inertial>
+  </link>
+  <joint name="airspeed_y_joint" type="fixed">
+    <parent link="base_link_front"/>
+    <child link="airspeed_y_link"/>
+    <origin xyz="0 0 0" rpy="0 0 1.5708"/>
+  </joint>
+  <!-- 5-hole probe vertical (body-z): sensor x-axis rotated to align with body +z -->
+  <link name="airspeed_z_link">
+    <inertial>
+      <mass value="0.001"/>
+      <origin xyz="-1.1 0 0.15"/>
+      <inertia ixx="1e-7" iyy="1e-7" izz="1e-7" ixy="0" ixz="0" iyz="0"/>
+    </inertial>
+  </link>
+  <joint name="airspeed_z_joint" type="fixed">
+    <parent link="base_link_front"/>
+    <child link="airspeed_z_link"/>
+    <origin xyz="0 0 0" rpy="0 -1.5708 0"/>
+  </joint>
   <link name="baro_link">
     <inertial>
@@ -483,5 +509,5 @@
       <inertia ixx="1e-5" ixy="0" ixz="0" iyy="1e-5" iyz="0" izz="1e-5"/>
     </inertial>
-    <collision><origin xyz="0 0 0"/><geometry><cylinder length="0.1" radius="0.015"/></geometry></collision>
+    <!-- NO COLLISION — spinning collision geometry causes ODE AABB overflow at high RPM -->
     <visual name="thruster_L_visual">
       <origin xyz="0 0 0" rpy="0 0 0"/>
@@ -498,5 +524,5 @@
       <inertia ixx="1e-5" ixy="0" ixz="0" iyy="1e-5" iyz="0" izz="1e-5"/>
     </inertial>
-    <collision><origin xyz="0 0 0"/><geometry><cylinder length="0.1" radius="0.015"/></geometry></collision>
+    <!-- NO COLLISION — spinning collision geometry causes ODE AABB overflow at high RPM -->
     <visual name="thruster_R_visual">
       <origin xyz="0 0 0" rpy="0 0 0"/>
@@ -510,6 +536,6 @@
     <parent link="base_link_front"/>
     <child  link="thruster_L"/>
-    <origin xyz="-1.20 -0.3 0.50" rpy="0 0 0"/>
-    <axis xyz="1 0 0"/>  <!-- Reverted: Original axis was correct -->
+    <origin xyz="-1.876 -0.3 0.306" rpy="0 0 0"/>
+    <axis xyz="1 0 0"/>
     <!-- Continuous joints don't have limits - unlimited rotation for propellers -->
     <dynamics damping="0.0" friction="0.0"/>  <!-- Zero damping to allow full reaction torque visibility -->
@@ -518,6 +544,6 @@
     <parent link="base_link_front"/>
     <child  link="thruster_R"/>
-    <origin xyz="-1.20 0.3 0.50" rpy="0 0 0"/>
-    <axis xyz="1 0 0"/>  <!-- Normal axis: both axes same, counter-rotation via negative angular velocity -->
+    <origin xyz="-1.876 0.3 0.306" rpy="0 0 0"/>
+    <axis xyz="1 0 0"/>
     <!-- Continuous joints don't have limits - unlimited rotation for propellers -->
     <dynamics damping="0.0" friction="0.0"/>  <!-- Zero damping to allow full reaction torque visibility -->
@@ -613,21 +639,3 @@
     <origin xyz="-0.5 0 0.1" rpy="0 1.5708 0"/>
   </joint>
-    <!-- Nose propeller (MulticopterMotorModel: command motor speed rad/s on command/motor_speed_nose) -->
-  <link name="nose_prop">
-    <inertial>
-      <origin xyz="-1.876 0 0.306" rpy="0 0 0"/>
-      <mass value="0.05"/>
-      <inertia ixx="5e-4" ixy="0" ixz="0" iyy="5e-4" iyz="0" izz="5e-4"/>
-    </inertial>
-    <visual>
-      <origin xyz="0 0 0.2" rpy="0 0 0"/>
-      <geometry><cylinder length="0.2" radius="0.015"/></geometry>
-    </visual>
-  </link>
-  <joint name="nose_prop_joint" type="continuous">
-    <parent link="base_link_front"/>
-    <child link="nose_prop"/>
-    <origin xyz="0 0 0.2" rpy="0 0 0"/>
-    <axis xyz="1 0 0"/>  <!-- Spin about X (body forward); thrust along +X -->
-  </joint>
 </robot>

File: src/marid_description/urdf/marid_new_gazebo.xacro (robot description, xacro)
@@ -181,14 +181,14 @@
             <zDotW>-1.2</zDotW>    <!-- Vertical drag (Z-axis) -->
             <!-- Angular drag - increased for larger vehicle -->
-            <kDotP>-4.0</kDotP>    <!-- Roll damping (around X) -->
-            <mDotQ>-4.0</mDotQ>    <!-- Pitch damping (around Y) -->
-            <nDotR>-4.0</nDotR>    <!-- Yaw damping (around Z) -->
+            <kDotP>-4.6</kDotP>    <!-- Roll damping (around X) — +15% from -4.0 -->
+            <mDotQ>-4.6</mDotQ>    <!-- Pitch damping (around Y) — +15% from -4.0 -->
+            <nDotR>-4.6</nDotR>    <!-- Yaw damping (around Z) — +15% from -4.0 -->
             <!-- Quadratic drag (velocity-squared) -->
             <xUabsU>-0.12</xUabsU>   <!-- Forward (X) quadratic drag -->
             <yVabsV>-0.35</yVabsV>   <!-- Lateral (Y) quadratic drag -->
             <zWabsW>-0.4</zWabsW>    <!-- Vertical quadratic drag -->
-            <kPabsP>-2.0</kPabsP>    <!-- Roll quadratic damping -->
-            <mQabsQ>-2.0</mQabsQ>    <!-- Pitch quadratic damping -->
-            <nRabsR>-2.0</nRabsR>    <!-- Yaw quadratic damping -->
+            <kPabsP>-2.3</kPabsP>    <!-- Roll quadratic damping — +15% from -2.0 -->
+            <mQabsQ>-2.3</mQabsQ>    <!-- Pitch quadratic damping — +15% from -2.0 -->
+            <nRabsR>-2.3</nRabsR>    <!-- Yaw quadratic damping — +15% from -2.0 -->
             <!-- Linear velocity terms (X-forward) -->
             <xU>-1.5</xU>         <!-- forward (X) -->
@@ -211,10 +211,11 @@
         </plugin>
     </gazebo>
-    <!-- ===== LEFT/RIGHT: Thruster plugin (force in Newtons) ===== -->
+    <!-- ===== LEFT/RIGHT: Dual thruster pair (prop diameter 0.35 m for realistic RPM at cruise) ===== -->
     <gazebo>
         <plugin filename="libgz-sim8-thruster-system.so" name="gz::sim::systems::Thruster">
             <joint_name>thruster_L_joint</joint_name>
             <fluid_density>1.204</fluid_density>
-            <propeller_diameter>0.08</propeller_diameter>
+            <propeller_diameter>0.35</propeller_diameter>
+            <thrust_coefficient>1.0</thrust_coefficient>
             <max_thrust_cmd>5000</max_thrust_cmd>
             <min_thrust_cmd>0</min_thrust_cmd>
@@ -225,31 +226,17 @@
             <joint_name>thruster_R_joint</joint_name>
             <fluid_density>1.204</fluid_density>
-            <propeller_diameter>0.08</propeller_diameter>
-            <max_thrust_cmd>5000</max_thrust_cmd>
-            <min_thrust_cmd>0</min_thrust_cmd>
-        </plugin>
-    </gazebo>
-    <!-- ===== NOSE PROPELLER: MulticopterMotorModel (motor speed rad/s) ===== -->
-    <!-- Topic: /model/marid/command/motor_speed_nose (gz.msgs.Double) -->
-    <gazebo>
-        <plugin name="gz::sim::systems::MulticopterMotorModel" filename="gz-sim-multicopter-motor-model-system">
-            <jointName>nose_prop_joint</jointName>
-            <linkName>nose_prop</linkName>
-            <turningDirection>cw</turningDirection>
-            <timeConstantUp>0.0125</timeConstantUp>
-            <timeConstantDown>0.025</timeConstantDown>
-            <maxRotVelocity>80000</maxRotVelocity>
-            <motorConstant>8.54858e-06</motorConstant>
-            <momentConstant>0.01</momentConstant>
-            <commandSubTopic>command/motor_speed_nose</commandSubTopic>
-            <motorNumber>0</motorNumber>
-            <rotorDragCoefficient>8.06428e-05</rotorDragCoefficient>
-            <rollingMomentCoefficient>1e-06</rollingMomentCoefficient>
-            <rotorVelocitySlowdownSim>10</rotorVelocitySlowdownSim>
-            <motorType>velocity</motorType>
+            <propeller_diameter>0.35</propeller_diameter>
+            <thrust_coefficient>1.0</thrust_coefficient>
+            <max_thrust_cmd>0</max_thrust_cmd>
+            <min_thrust_cmd>-5000</min_thrust_cmd>
         </plugin>
     </gazebo>
     <!-- ===== JOINT POSITION CONTROLLERS FOR CONTROL SURFACES ===== -->
-    <!-- P-gain chosen so controllers can hold wings/tails stiff against aero and gravity with ~10 N·m joint friction -->
+    <!-- PID tuned for servo-like disturbance rejection:
+         - P provides immediate corrective torque (stiffness)
+         - I nulls steady-state aero hinge moments (the "locked" behavior)
+         - D damps velocity-based disturbances during aggressive maneuvers
+         Coulomb friction in the URDF is intentionally NOT increased because it resists
+         commanded motion equally — PID active holding is the right mechanism. -->
     <!-- Left Wing Position Controller -->
     <gazebo>
@@ -257,5 +244,11 @@
                 name="gz::sim::systems::JointPositionController">
             <joint_name>left_wing_joint</joint_name>
-            <p_gain>600.0</p_gain>
+            <p_gain>4000.0</p_gain>
+            <i_gain>5.0</i_gain>
+            <d_gain>80.0</d_gain>
+            <i_max>200.0</i_max>
+            <i_min>-200.0</i_min>
+            <cmd_max>1500.0</cmd_max>
+            <cmd_min>-1500.0</cmd_min>
             <topic>/model/marid/joint/left_wing_joint/cmd_pos</topic>
         </plugin>
@@ -266,5 +259,11 @@
                 name="gz::sim::systems::JointPositionController">
             <joint_name>right_wing_joint</joint_name>
-            <p_gain>600.0</p_gain>
+            <p_gain>4000.0</p_gain>
+            <i_gain>5.0</i_gain>
+            <d_gain>80.0</d_gain>
+            <i_max>200.0</i_max>
+            <i_min>-200.0</i_min>
+            <cmd_max>1500.0</cmd_max>
+            <cmd_min>-1500.0</cmd_min>
             <topic>/model/marid/joint/right_wing_joint/cmd_pos</topic>
         </plugin>
@@ -275,5 +274,11 @@
                 name="gz::sim::systems::JointPositionController">
             <joint_name>tail_left_joint</joint_name>
-            <p_gain>280.0</p_gain>
+            <p_gain>2500.0</p_gain>
+            <i_gain>3.0</i_gain>
+            <d_gain>50.0</d_gain>
+            <i_max>100.0</i_max>
+            <i_min>-100.0</i_min>
+            <cmd_max>1000.0</cmd_max>
+            <cmd_min>-1000.0</cmd_min>
             <topic>/model/marid/joint/tail_left_joint/cmd_pos</topic>
         </plugin>
@@ -284,5 +289,11 @@
                 name="gz::sim::systems::JointPositionController">
             <joint_name>tail_right_joint</joint_name>
-            <p_gain>280.0</p_gain>
+            <p_gain>2500.0</p_gain>
+            <i_gain>3.0</i_gain>
+            <d_gain>50.0</d_gain>
+            <i_max>100.0</i_max>
+            <i_min>-100.0</i_min>
+            <cmd_max>1000.0</cmd_max>
+            <cmd_min>-1000.0</cmd_min>
             <topic>/model/marid/joint/tail_right_joint/cmd_pos</topic>
         </plugin>
@@ -300,5 +311,5 @@
                 <noise type="gaussian">
                   <mean>0.0</mean>
-                  <stddev>2e-4</stddev>
+                  <stddev>2e-6</stddev> <!-- FOG/RLG-like low angular-rate noise -->
                 </noise>
               </x>
@@ -306,5 +317,5 @@
                 <noise type="gaussian">
                   <mean>0.0</mean>
-                  <stddev>2e-4</stddev>
+                  <stddev>2e-6</stddev> <!-- FOG/RLG-like low angular-rate noise -->
                 </noise>
               </y>
@@ -312,5 +323,5 @@
                 <noise type="gaussian">
                   <mean>0.0</mean>
-                  <stddev>2e-4</stddev>
+                  <stddev>2e-6</stddev> <!-- FOG/RLG-like low angular-rate noise -->
                 </noise>
               </z>
@@ -320,5 +331,5 @@
                 <noise type="gaussian">
                   <mean>0.0</mean>
-                  <stddev>1.7e-2</stddev>
+                  <stddev>2e-3</stddev>
                 </noise>
               </x>
@@ -326,5 +337,5 @@
                 <noise type="gaussian">
                   <mean>0.0</mean>
-                  <stddev>1.7e-2</stddev>
+                  <stddev>2e-3</stddev>
                 </noise>
               </y>
@@ -332,5 +343,5 @@
                 <noise type="gaussian">
                   <mean>0.0</mean>
-                  <stddev>1.7e-2</stddev>
+                  <stddev>2e-3</stddev>
                 </noise>
               </z>
@@ -353,5 +364,5 @@
               <noise type="gaussian">
                 <mean>0.0</mean>
-                <stddev>0.00002</stddev> <!-- ~2.5m equiv (workaround for degrees bug) -->
+                <stddev>0.000002</stddev> <!-- ~0.25m equiv (workaround for degrees bug) -->
               </noise>
             </horizontal>
@@ -359,5 +370,5 @@
               <noise type="gaussian">
                 <mean>0.0</mean>
-                <stddev>0.00002</stddev> <!-- ~2.5m equiv (workaround for degrees bug) -->
+                <stddev>0.000002</stddev> <!-- ~0.25m equiv (workaround for degrees bug) -->
               </noise>
             </vertical>
@@ -368,5 +379,5 @@
               <noise type="gaussian">
                 <mean>0.0</mean>
-                <stddev>1.5</stddev> <!-- 0.1 m/s velocity accuracy -->
+                <stddev>0.05</stddev> <!-- high-quality Doppler velocity accuracy -->
               </noise>
             </horizontal>
@@ -374,5 +385,5 @@
               <noise type="gaussian">
                 <mean>0.0</mean>
-                <stddev>1.5</stddev>
+                <stddev>0.05</stddev>
               </noise>
             </vertical>
@@ -412,5 +423,5 @@
             <type>gaussian</type>
             <mean>0.0</mean>
-            <stddev>0.01</stddev>  <!-- 1 cm standard deviation -->
+            <stddev>0.002</stddev>  <!-- 2 mm standard deviation -->
           </noise>
         </ray>
@@ -431,5 +442,5 @@
             <noise type="gaussian">
               <mean>0.0</mean>
-              <stddev>5e-8</stddev>
+              <stddev>1e-8</stddev>
             </noise>
           </x>
@@ -437,5 +448,5 @@
             <noise type="gaussian">
               <mean>0.0</mean>
-              <stddev>5e-8</stddev>
+              <stddev>1e-8</stddev>
             </noise>
           </y>
@@ -443,5 +454,5 @@
             <noise type="gaussian">
               <mean>0.0</mean>
-              <stddev>5e-8</stddev>
+              <stddev>1e-8</stddev>
             </noise>
           </z>
@@ -458,5 +469,5 @@
             <noise type="gaussian">
               <mean>0.0</mean>
-              <stddev>0.1</stddev> <!-- 0.1 m/s accuracy -->
+              <stddev>0.01</stddev>
             </noise>
           </pressure>
@@ -464,4 +475,34 @@
       </sensor>
     </gazebo>
+    <gazebo reference="airspeed_y_link">
+      <sensor name="airspeed_y" type="air_speed">
+        <always_on>true</always_on>
+        <update_rate>50</update_rate>
+        <topic>/airspeed_y</topic>
+        <air_speed>
+          <pressure>
+            <noise type="gaussian">
+              <mean>0.0</mean>
+              <stddev>0.01</stddev>
+            </noise>
+          </pressure>
+        </air_speed>
+      </sensor>
+    </gazebo>
+    <gazebo reference="airspeed_z_link">
+      <sensor name="airspeed_z" type="air_speed">
+        <always_on>true</always_on>
+        <update_rate>50</update_rate>
+        <topic>/airspeed_z</topic>
+        <air_speed>
+          <pressure>
+            <noise type="gaussian">
+              <mean>0.0</mean>
+              <stddev>0.01</stddev>
+            </noise>
+          </pressure>
+        </air_speed>
+      </sensor>
+    </gazebo>
     <gazebo reference="baro_link">
       <sensor name="baro" type="air_pressure">
@@ -471,5 +512,5 @@
         <noise type="gaussian">
           <mean>0.0</mean>
-          <stddev>0.5</stddev>
+          <stddev>0.05</stddev>
         </noise>
       </sensor>
@@ -497,5 +538,5 @@
             <type>gaussian</type>
             <mean>0.0</mean>
-            <stddev>1.5</stddev>
+            <stddev>0.1</stddev>
           </noise>
         </camera>
@@ -533,5 +574,5 @@
             <type>gaussian</type>
             <mean>0.0</mean>
-            <stddev>0.02</stddev>
+            <stddev>0.005</stddev>
           </noise>
         </ray>
